File: PCB/SRAM_XC7A100T.kicad_sch (KiCad schematic)
At the start: 0 parts

Commit message: pcb: cleanup mcu sram (#10)
Co-authored-by: Kolbjørn Austreng <kolbjorn.austreng@hotzen.io>
Parts:
- added C28: 0.1u, symbol Device:C_Small
- added U7: IS62WVS2568FBLL-20NLI, symbol 0000_CustomComponents:IS62WVS2568FBLL-20NLI-TR | SQI Mode
Connections:
- new net +3.3V: C28.1, U7.8 (VCC)
- new net CLK: U7.6 (SCK)
- new net GND: C28.2, U7.4 (VSS)
- new net IO0: U7.5 (SIO0)
- new net IO1: U7.2 (SIO1)
- new net IO2: U7.3 (SIO2)
- new net IO3: U7.7 (SIO3)
- new net SS: U7.1 (CS#)
Other:
- note added: "The device starts in SPI mode, execute the ESQI (0x38) command to enter QSPI mode."
Changed lines of the file:
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@@
 (kicad_sch (version 20230121) (generator eeschema)
   (paper "A4")
+  (junction (at 154.94 82.55) (diameter 0) (color 0 0 0 0)
+  )
+  (wire (pts (xy 154.94 82.55) (xy 154.94 86.36))
+    (stroke (width 0) (type default))
+  )
+  (wire (pts (xy 92.71 87.63) (xy 101.6 87.63))
+    (stroke (width 0) (type default))
+  )
+  (wire (pts (xy 99.06 95.25) (xy 99.06 90.17))
+    (stroke (width 0) (type default))
+  )
+  (wire (pts (xy 127 82.55) (xy 154.94 82.55))
+    (stroke (width 0) (type default))
+  )
+  (wire (pts (xy 135.89 90.17) (xy 127 90.17))
+    (stroke (width 0) (type default))
+  )
+  (wire (pts (xy 92.71 82.55) (xy 101.6 82.55))
+    (stroke (width 0) (type default))
+  )
+  (wire (pts (xy 160.02 74.93) (xy 160.02 82.55))
+    (stroke (width 0) (type default))
+  )
+  (wire (pts (xy 135.89 87.63) (xy 127 87.63))
+    (stroke (width 0) (type default))
+  )
+  (wire (pts (xy 99.06 90.17) (xy 101.6 90.17))
+    (stroke (width 0) (type default))
+  )
+  (wire (pts (xy 154.94 82.55) (xy 160.02 82.55))
+    (stroke (width 0) (type default))
+  )
+  (wire (pts (xy 92.71 85.09) (xy 101.6 85.09))
+    (stroke (width 0) (type default))
+  )
+  (wire (pts (xy 154.94 91.44) (xy 154.94 95.25))
+    (stroke (width 0) (type default))
+  )
+  (wire (pts (xy 135.89 85.09) (xy 127 85.09))
+    (stroke (width 0) (type default))
+  )
+  (text "The device starts in SPI mode,\nexecute the ESQI (0x38) command\nto enter QSPI mode."
+    (at 99.06 69.85 0)
+    (effects (font (size 1.27 1.27)) (justify left bottom))
+  )
+  (hierarchical_label "IO2" (shape bidirectional) (at 92.71 87.63 180) (fields_autoplaced)
+    (effects (font (size 1.27 1.27)) (justify right))
+  )
+  (hierarchical_label "IO0" (shape bidirectional) (at 135.89 90.17 0) (fields_autoplaced)
+    (effects (font (size 1.27 1.27)) (justify left))
+  )
+  (hierarchical_label "CLK" (shape input) (at 135.89 87.63 0) (fields_autoplaced)
+    (effects (font (size 1.27 1.27)) (justify left))
+  )
+  (hierarchical_label "IO3" (shape bidirectional) (at 135.89 85.09 0) (fields_autoplaced)
+    (effects (font (size 1.27 1.27)) (justify left))
+  )
+  (hierarchical_label "SS" (shape input) (at 92.71 82.55 180) (fields_autoplaced)
+    (effects (font (size 1.27 1.27)) (justify right))
+  )
+  (hierarchical_label "IO1" (shape bidirectional) (at 92.71 85.09 180) (fields_autoplaced)
+    (effects (font (size 1.27 1.27)) (justify right))
+  )
+  (symbol (lib_id "power:+3.3V") (at 160.02 74.93 0) (unit 1)
+    (in_bom yes) (on_board yes) (dnp no) (fields_autoplaced)
+    (property "Reference" "#PWR017" (at 160.02 78.74 0)
+      (effects (font (size 1.27 1.27)) hide)
+    )
+    (property "Value" "+3.3V" (at 160.02 69.85 0)
+      (effects (font (size 1.27 1.27)))
+    )
+    (property "Footprint" "" (at 160.02 74.93 0)
+      (effects (font (size 1.27 1.27)) hide)
+    )
+    (property "Datasheet" "" (at 160.02 74.93 0)
+      (effects (font (size 1.27 1.27)) hide)
+    )
+    (pin "1")
+    (instances
+      (project "RayTracingPCB"
+        (path "/e9047d94-28be-4266-894b-6ee25ef088bd/f9a74965-bde5-47a2-9f66-243cb6fc0f53"
+          (reference "#PWR017") (unit 1)
+        )
+        (path "/e9047d94-28be-4266-894b-6ee25ef088bd/e35285fd-162a-4f7e-974b-e69dceb1cfdc"
+          (reference "#PWR022") (unit 1)
+        )
+        (path "/e9047d94-28be-4266-894b-6ee25ef088bd/5a7a2c0a-f09d-4b4f-9411-f51dd121457c/65904ece-fe30-45bb-94bd-e245ab68e3ab"
+          (reference "#PWR027") (unit 1)
+        )
+      )
+    )
+  )
+  (symbol (lib_id "power:GND") (at 99.06 95.25 0) (unit 1)
+    (in_bom yes) (on_board yes) (dnp no) (fields_autoplaced)
+    (property "Reference" "#PWR014" (at 99.06 101.6 0)
+      (effects (font (size 1.27 1.27)) hide)
+    )
+    (property "Value" "GND" (at 99.06 100.33 0)
+      (effects (font (size 1.27 1.27)))
+    )
+    (property "Footprint" "" (at 99.06 95.25 0)
+      (effects (font (size 1.27 1.27)) hide)
+    )
+    (property "Datasheet" "" (at 99.06 95.25 0)
+      (effects (font (size 1.27 1.27)) hide)
+    )
+    (pin "1")
+    (instances
+      (project "RayTracingPCB"
+        (path "/e9047d94-28be-4266-894b-6ee25ef088bd/5a7a2c0a-f09d-4b4f-9411-f51dd121457c/3d4f3bb6-8d8f-4b26-b7c8-e791b7e32814"
+          (reference "#PWR014") (unit 1)
+        )
+        (path "/e9047d94-28be-4266-894b-6ee25ef088bd/e35285fd-162a-4f7e-974b-e69dceb1cfdc"
+          (reference "#PWR023") (unit 1)
+        )
+        (path "/e9047d94-28be-4266-894b-6ee25ef088bd/5a7a2c0a-f09d-4b4f-9411-f51dd121457c/65904ece-fe30-45bb-94bd-e245ab68e3ab"
+          (reference "#PWR025") (unit 1)
+        )
+      )
+    )
+  )
+  (symbol (lib_id "0000_CustomComponents:IS62WVS2568FBLL-20NLI-TR | SQI Mode") (at 114.3 78.74 0) (unit 1)
+    (in_bom yes) (on_board yes) (dnp no)
+    (property "Reference" "U7" (at 114.2093 74.93 0)
+      (effects (font (size 1.27 1.27)))
+    )
+    (property "Value" "IS62WVS2568FBLL-20NLI" (at 114.2093 77.47 0)
+      (effects (font (size 1.27 1.27)))
+    )
+    (property "Footprint" "" (at 114.3 78.74 0)
+      (effects (font (size 1.27 1.27)) hide)
+    )
+    (property "Datasheet" "https://www.issi.com/WW/pdf/IS62-65WVS2568FALL-BLL.pdf" (at 114.3 78.74 0)
+      (effects (font (size 1.27 1.27)) hide)
+    )
+    (pin "1")
+    (pin "2")
+    (pin "3")
+    (pin "4")
+    (pin "5")
+    (pin "6")
+    (pin "7")
+    (pin "8")
+    (instances
+      (project "RayTracingPCB"
+        (path "/e9047d94-28be-4266-894b-6ee25ef088bd/e35285fd-162a-4f7e-974b-e69dceb1cfdc"
+          (reference "U7") (unit 1)
+        )
+        (path "/e9047d94-28be-4266-894b-6ee25ef088bd/5a7a2c0a-f09d-4b4f-9411-f51dd121457c/65904ece-fe30-45bb-94bd-e245ab68e3ab"
+          (reference "U6") (unit 1)
+        )
+      )
+    )
+  )
+  (symbol (lib_id "power:GND") (at 154.94 95.25 0) (unit 1)
+    (in_bom yes) (on_board yes) (dnp no) (fields_autoplaced)
+    (property "Reference" "#PWR014" (at 154.94 101.6 0)
+      (effects (font (size 1.27 1.27)) hide)
+    )
+    (property "Value" "GND" (at 154.94 100.33 0)
+      (effects (font (size 1.27 1.27)))
+    )
+    (property "Footprint" "" (at 154.94 95.25 0)
+      (effects (font (size 1.27 1.27)) hide)
+    )
+    (property "Datasheet" "" (at 154.94 95.25 0)
+      (effects (font (size 1.27 1.27)) hide)
+    )
+    (pin "1")
+    (instances
+      (project "RayTracingPCB"
+        (path "/e9047d94-28be-4266-894b-6ee25ef088bd/5a7a2c0a-f09d-4b4f-9411-f51dd121457c/3d4f3bb6-8d8f-4b26-b7c8-e791b7e32814"
+          (reference "#PWR014") (unit 1)
+        )
+        (path "/e9047d94-28be-4266-894b-6ee25ef088bd/e35285fd-162a-4f7e-974b-e69dceb1cfdc"
+          (reference "#PWR024") (unit 1)
+        )
+        (path "/e9047d94-28be-4266-894b-6ee25ef088bd/5a7a2c0a-f09d-4b4f-9411-f51dd121457c/65904ece-fe30-45bb-94bd-e245ab68e3ab"
+          (reference "#PWR026") (unit 1)
+        )
+      )
+    )
+  )
+  (symbol (lib_id "Device:C_Small") (at 154.94 88.9 0) (unit 1)
+    (in_bom yes) (on_board yes) (dnp no) (fields_autoplaced)
+    (property "Reference" "C28" (at 157.48 87.6363 0)
+      (effects (font (size 1.27 1.27)) (justify left))
+    )
+    (property "Value" "0.1u" (at 157.48 90.1763 0)
+      (effects (font (size 1.27 1.27)) (justify left))
+    )
+    (property "Footprint" "" (at 154.94 88.9 0)
+      (effects (font (size 1.27 1.27)) hide)
+    )
+    (property "Datasheet" "~" (at 154.94 88.9 0)
+      (effects (font (size 1.27 1.27)) hide)
+    )
+    (pin "1")
+    (pin "2")
+    (instances
+      (project "RayTracingPCB"
+        (path "/e9047d94-28be-4266-894b-6ee25ef088bd/e35285fd-162a-4f7e-974b-e69dceb1cfdc"
+          (reference "C28") (unit 1)
+        )
+        (path "/e9047d94-28be-4266-894b-6ee25ef088bd/5a7a2c0a-f09d-4b4f-9411-f51dd121457c/65904ece-fe30-45bb-94bd-e245ab68e3ab"
+          (reference "C27") (unit 1)
+        )
+      )
+    )
+  )
 )
