File: PCB/VGA.kicad_sch (KiCad schematic)
At the start: 0 parts

Commit message: dump
Parts:
- added C30: 1nF, symbol Device:C_Small
- added J2: DE15_Plug_HighDensity_MountingHoles, Connector_Dsub:DSUB-15-HD_Female_Horizontal_P2.29x1.98mm_EdgePinOffset3.03mm_Housed_MountingHolesOffset4.94mm, symbol Connector:DE15_Plug_HighDensity_MountingHoles
- added R14, R15: 100, symbol Device:R_Small
- added R16: 1M, symbol Device:R_Small
- added R17, R28, R32: 2k, symbol Device:R_Small
- added R23, R26, R30: 4k, symbol Device:R_Small
- added R24, R29, R33: 510, symbol Device:R_Small
- added R25, R27, R31: 1K, symbol Device:R_Small
Connections:
- new net: J2.3, R26.2, R27.2, R28.2, R29.2
- new net: J2.2, R30.2, R31.2, R32.2, R33.2
- new net: J2.13, R15.1
- new net: J2.1, R17.2, R23.2, R24.2, R25.2
- new net: C30.1, J2.0, R16.1
- new net: J2.14, R14.1
- new net GND: C30.2, J2.10, J2.5, J2.6, J2.7, J2.8, R16.2
- new net VGA_B0: R26.1
- new net VGA_B1: R28.1
- new net VGA_B2: R27.1
- new net VGA_B3: R29.1
- new net VGA_G0: R30.1
- new net VGA_G1: R32.1
- new net VGA_G2: R31.1
- new net VGA_G3: R33.1
- new net VGA_HSync: R14.2
- new net VGA_R0: R23.1
- new net VGA_R1: R17.1
- new net VGA_R2: R25.1
- new net VGA_R3: R24.1
- new net VGA_VSync: R15.2
- no-connect marks 0 -> 2
