File: PCB/TripSitter/FPGA_bank34_ddr3.kicad_sch (KiCad schematic)
At the start: 13 parts, among them IC2 MT41J128M16JT-125_K, U1 XC7A100T-FGG484, X1 XO53 100Mhz

Commit message: attempt at routing
Parts:
- removed C29, C97: 0.1uF, Capacitor_SMD:C_0201_0603Metric_Pad0.64x0.40mm_HandSolder, symbol Device:C_Small
- removed C99: 100uF, Capacitor_SMD:C_0805_2012Metric_Pad1.18x1.45mm_HandSolder, symbol Device:C_Small
- removed unit 3 of U1
- added R41: 100R, symbol Device:R_Small
- IC2: footprint footprints:FBGA96_8X14_MRN -> Package_BGA:Micron_FBGA-96_8x14mm_Layout9x16_P0.8mm
Connections:
- net DDR3_A0: now also U1.AB5 (IO_L10N_T1_34); no longer U1.W5 (IO_L15N_T2_DQS_34)
- net DDR3_A1: now also U1.Y6 (IO_L18P_T2_34); no longer U1.T6 (IO_L17N_T2_34)
- net DDR3_A10: now also U1.AB6 (IO_L20N_T3_34); no longer U1.Y6 (IO_L18P_T2_34)
- net DDR3_A11: now also U1.AB7 (IO_L20P_T3_34); no longer U1.AB8 (IO_L22N_T3_34)
- net DDR3_A12: now also U1.AA6 (IO_L18N_T2_34); no longer U1.Y7 (IO_L23N_T3_34)
- net DDR3_A13: now also U1.AB1 (IO_L7N_T1_34); no longer U1.Y9 (IO_L24N_T3_34)
- net DDR3_A2: now also U1.AB3 (IO_L8P_T1_34); no longer U1.V5 (IO_L16N_T2_34)
- net DDR3_A3: now also U1.U1 (IO_L1N_T0_34); no longer U1.V7 (IO_L19P_T3_34)
- net DDR3_A4: now also U1.Y9 (IO_L24N_T3_34); no longer U1.W7 (IO_L19N_T3_VREF_34)
- net DDR3_A5: now also U1.W1 (IO_L5P_T0_34); no longer U1.Y8 (IO_L23P_T3_34)
- net DDR3_A6: now also U1.AA8 (IO_L22P_T3_34); no longer U1.AB6 (IO_L20N_T3_34)
- net DDR3_A7: now also U1.Y1 (IO_L5N_T0_34); no longer U1.AA8 (IO_L22P_T3_34)
- net DDR3_A8: now also U1.AB8 (IO_L22N_T3_34); no longer U1.W9 (IO_L24P_T3_34)
- net DDR3_A9: now also U1.AB2 (IO_L8N_T1_34); no longer U1.AA6 (IO_L18N_T2_34)
- net DDR3_BA0: now also U1.T1 (IO_L1P_T0_34); no longer U1.R6 (IO_L17P_T2_34)
- net DDR3_BA1: now also U1.W9 (IO_L24P_T3_34); no longer U1.T5 (IO_L14P_T2_SRCC_34)
- net DDR3_BA2: now also U1.AA4 (IO_L11N_T1_SRCC_34); no longer U1.W6 (IO_L15P_T2_DQS_34)
- net DDR3_DQ0: now also U1.Y8 (IO_L23P_T3_34); no longer U1.W1 (IO_L5P_T0_34)
- net DDR3_DQ10: now also U1.V5 (IO_L16N_T2_34); no longer U1.AB3 (IO_L8P_T1_34)
- net DDR3_DQ11: now also U1.T5 (IO_L14P_T2_SRCC_34); no longer U1.AA5 (IO_L10P_T1_34)
- net DDR3_DQ12: now also U1.W6 (IO_L15P_T2_DQS_34); no longer U1.AB1 (IO_L7N_T1_34)
- net DDR3_DQ13: now also U1.W7 (IO_L19N_T3_VREF_34); no longer U1.AA4 (IO_L11N_T1_SRCC_34)
- net DDR3_DQ14: now also U1.AA5 (IO_L10P_T1_34); no longer U1.AB2 (IO_L8N_T1_34)
- net DDR3_DQ5: now also U1.V7 (IO_L19P_T3_34); no longer U1.U1 (IO_L1N_T0_34)
- net DDR3_DQ6: now also U1.T3 (IO_0_34); no longer U1.Y1 (IO_L5N_T0_34)
- net DDR3_DQ8: now also U1.W5 (IO_L15N_T2_DQS_34); no longer U1.AB5 (IO_L10N_T1_34)
- net DDR3_LDM: now also U1.Y7 (IO_L23N_T3_34); no longer U1.T1 (IO_L1P_T0_34)
- net DDR3_ODT: now also U1.T6 (IO_L17N_T2_34); no longer U1.AB7 (IO_L20P_T3_34)
- net DDR3_UDM: now also U1.R6 (IO_L17P_T2_34); no longer U1.AA1 (IO_L7P_T1_34)
- net DDR3_nRESET: now also U1.AA1 (IO_L7P_T1_34); no longer U1.T3 (IO_0_34)
- net XO_Enable: now also U1.V3 (IO_L6N_T0_VREF_34)
- removed net DDR3_A14: IC2.N7 (A14), U1.V3 (IO_L6N_T0_VREF_34)
- net DDR3_CK renamed DDR3_CK_N
- net DDR3_CK_N: now also IC2.K7 (CK#), R41.2; no longer IC2.J7 (CK)
- net DDR3_LDQS renamed DDR3_LDQS_P
- net DDR3_UDQS renamed DDR3_UDQS_N
- net DDR3_UDQS_N: now also IC2.B7 (UDQS#); no longer IC2.C7 (UDQS)
- net DDR3_nCK renamed DDR3_CK_P
- net DDR3_CK_P: now also IC2.J7 (CK), R41.1; no longer IC2.K7 (CK#)
- net DDR3_nLDQS renamed DDR3_LDQS_N
- net DDR3_nUDQS renamed DDR3_UDQS_P
- net DDR3_UDQS_P: now also IC2.C7 (UDQS); no longer IC2.B7 (UDQS#)
Other:
- note added: "Capacitor placement guide Ref. https://www.micron.com/-/media/client/global/documents/products/technical-note/dram/tn4113_ddr3_point_to_point_design.pdf"
- note added: "We don't need to route A14 for 2GB"
