File: PCB/TripSitter/FPGA_bank34_ddr3.kicad_sch (KiCad schematic)
At the start: 11 parts, among them IC2 MT41J128M16JT-125_K, U1 XC7A100T-FGG484, X1 XO53 100Mhz

Commit message: before
Parts:
- removed C25, C26: 0.1uF, Capacitor_SMD:C_0201_0603Metric_Pad0.64x0.40mm_HandSolder, symbol Device:C_Small
- removed C27: 100uF, Capacitor_SMD:C_0805_2012Metric_Pad1.18x1.45mm_HandSolder, symbol Device:C_Small
- removed R41: 100R, symbol Device:R_Small
- added C16: 100uF, Capacitor_SMD:C_1210_3225Metric_Pad1.33x2.70mm_HandSolder, symbol Device:C_Small
- added C19: 47uF, Capacitor_SMD:C_1210_3225Metric_Pad1.33x2.70mm_HandSolder, symbol Device:C_Small
- added C20 (x2): 4.7uF, Capacitor_SMD:C_0805_2012Metric_Pad1.18x1.45mm_HandSolder, symbol Device:C_Small
- added R804: 100R, Resistor_SMD:R_0201_0603Metric_Pad0.64x0.40mm_HandSolder, symbol Device:R_Small
- IC2: Extra data (none) -> https://www.micron.com/-/media/client/global/documents/prod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
Connections:
- net +1V5: now also C16.1, C19.1, C20.1, C20.1
- net DDR3_CK_N: now also R804.2
- net DDR3_CK_P: now also R804.1
- net GND: now also C16.2, C19.2, C20.2, C20.2
Other:
- moved on the sheet: C94, C95, C96, IC2, R13, U1H, X1
