File: PCB/TripSitter/mcu_efm32gg11b420.kicad_sch (KiCad schematic)
At the start: 22 parts, among them J102 EFM32_PinHeader_PortE, J3 Conn_ARM_JTAG_SWD_20, SW1 SW_Push_Open, U3 IS62WVS2568FBLL-20NLI, U4 EFM32GG11B420F2048GQ100, Y101 48MHz

Commit message: before
Parts:
- removed C46, C47, C49, C52, C53, C57: 0.1uF, Capacitor_SMD:C_0201_0603Metric_Pad0.64x0.40mm_HandSolder, symbol Device:C_Small
- removed C54: 10uF, Capacitor_SMD:C_0402_1005Metric_Pad0.74x0.62mm_HandSolder, symbol Device:C_Small
- removed C55: 10nF, Capacitor_SMD:C_0402_1005Metric_Pad0.74x0.62mm_HandSolder, symbol Device:C_Small
- removed C59: 1uF, Capacitor_SMD:C_0201_0603Metric_Pad0.64x0.40mm_HandSolder, symbol Device:C_Small
- removed R19: 100k, Resistor_SMD:R_0805_2012Metric_Pad1.20x1.40mm_HandSolder, symbol Device:R_Small
- added C203, C204, C205, C206, C212, C213: 0.1uF, Capacitor_SMD:C_0603_1608Metric_Pad1.08x0.95mm_HandSolder, symbol Device:C_Small
- added C208: 10nF, Capacitor_SMD:C_0402_1005Metric_Pad0.74x0.62mm_HandSolder, symbol Device:C_Small
- added C209: 10uF, Capacitor_SMD:C_0402_1005Metric_Pad0.74x0.62mm_HandSolder, symbol Device:C_Small
- added C211: 1uF, Capacitor_SMD:C_0201_0603Metric_Pad0.64x0.40mm_HandSolder, symbol Device:C_Small
- added J102 (x4): EFM32_PinHeader_PortE, Connector_PinHeader_1.00mm:PinHeader_2x06_P1.00mm_Vertical, symbol Connector_Generic:Conn_02x06_Odd_Even
- added R804: 100K, Resistor_SMD:R_0805_2012Metric_Pad1.20x1.40mm_HandSolder, symbol Device:R
- C202: renamed from C51; footprint Capacitor_SMD:C_0201_0603Metric_Pad0.64x0.40mm_HandSolder -> Capacitor_SMD:C_0603_1608Metric_Pad1.08x0.95mm_HandSolder; Component Name (none) -> CL10B104KA8NNNC; DK_Ref (none) -> https://www.digikey.no/en/products/detail/samsung-electro-m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
- C210: renamed from C48; DK_Ref (none) -> https://www.digikey.no/no/products/detail/samsung-electro-m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; Digikey_ref https://www.digikey.no/no/products/detail/samsung-electro-m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 -> (none)
- J102: footprint Connector_PinHeader_2.54mm:PinHeader_2x06_P2.54mm_Vertical_SMD -> Connector_PinHeader_1.00mm:PinHeader_2x06_P1.00mm_Vertical
- SW1: footprint Button_Switch_SMD:SW_DIP_SPSTx01_Slide_6.7x4.1mm_W8.61mm_P2.54mm_LowProfile -> Button_Switch_SMD:SW_Push_1P1T_NO_CK_PTS125Sx43PSMTR
- renumbered C50 to C201, C56 to C207, C58 to C214, J3 to J201, U4 to U201, U3 to U202
Connections:
- net EBI_A27 is gone; now on net PC3: U201.68 (PC8)
- net EBI_A6 is gone; now on net EBI_AD10: U201.33 (PA12)
- net EBI_A7 is gone; now on net EBI_AD11: U201.34 (PA13)
- net EBI_A8 is gone; now on net EBI_AD12: U201.35 (PA14)
- net EBI_AD8 is gone; now on net EBI_AD9: U201.100 (PA15)
- net +3.3V: now also C203.1, C204.1, C205.1, C206.1, C212.1, C213.1, R804.1
- net +3.3VA: now also C208.2, C209.1
- net EBI_AD10: now also J102.8 (Pin_8); no longer U201.2 (PA1)
- net EBI_AD11: now also J102.10 (Pin_10); no longer U201.3 (PA2)
- net EBI_AD12: now also J102.12 (Pin_12); no longer U201.4 (PA3)
- net EBI_AD4: now also J102.9 (Pin_9)
- net EBI_AD5: now also J102.11 (Pin_11)
- net EBI_AD6: now also J102.4 (Pin_4)
- net EBI_AD7: now also J102.2 (Pin_2)
- net EBI_AD9: now also J102.6 (Pin_6); no longer U201.1 (PA0)
- net EFM32_RESETN: now also R804.2
- net GND: now also C203.2, C204.2, C205.2, C206.2, C208.1, C209.2, C211.2, C212.2, C213.2
- net PB10: now reaches U201.38 (PB10)
- net PB10: now also J102.6 (Pin_6)
- net PB11: now reaches U201.39 (PB11)
- net PB11: now also J102.5 (Pin_5)
- net PB12: now reaches U201.40 (PB12)
- net PB12: now also J102.7 (Pin_7)
- net at U201.73 (VREGO): now also C211.1
- net at U201.49 (PD3): now also J102.7 (Pin_7)
- net at U201.50 (PD4): now also J102.9 (Pin_9)
- net PC9: now reaches U201.69 (PC9)
- net PC9: now also J102.10 (Pin_10)
- net PC10: now reaches U201.70 (PC10)
- net PC10: now also J102.9 (Pin_9)
- net EBI_A0 renamed PB9
- net PB9: now also J102.4 (Pin_4)
- net EBI_A1 renamed PA7
- net PA7: now also J102.3 (Pin_3)
- net EBI_A10 renamed PD6
- net PD6: now also J102.2 (Pin_2)
- net EBI_A11 renamed PD7
- net PD7: now also J102.4 (Pin_4)
- net EBI_A12 renamed PD8
- net PD8: now also J102.6 (Pin_6)
- net EBI_A13: no longer names the net of U201.46 (PD0)
- net EBI_A13: now also J102.1 (Pin_1)
- net EBI_A14: no longer names the net of U201.47 (PD1)
- net EBI_A14: now also J102.3 (Pin_3)
- net EBI_A15: no longer names the net of U201.48 (PD2)
- net EBI_A15: now also J102.5 (Pin_5)
- net EBI_A16 renamed PB0
- net PB0: now also J102.1 (Pin_1)
- net EBI_A17 renamed PB1
- net PB1: now also J102.2 (Pin_2)
- net EBI_A18 renamed PB2
- net PB2: now also J102.3 (Pin_3)
- net EBI_A19 renamed QSPI0_DQ4
- net EBI_A2 renamed PA8
- net PA8: now also J102.5 (Pin_5)
- net EBI_A20 renamed QSPI0_DQ5
- net EBI_A21 renamed QSPI0_DQ6
- net EBI_A22 renamed QSPI0_DQ7
- net EBI_A23 renamed PC0
- net PC0: now also J102.8 (Pin_8)
- net EBI_A24 renamed PC1
- net PC1: now also J102.10 (Pin_10)
- net EBI_A25 renamed PC2
- net PC2: now also J102.12 (Pin_12)
- net EBI_A26 renamed PC3
- net PC3: now also J102.12 (Pin_12)
- net EBI_A3 renamed PA9
- net PA9: now also J102.7 (Pin_7)
- net EBI_A4 renamed PA10
- net PA10: now also J102.9 (Pin_9)
- net EBI_A5 renamed PA11
- net PA11: now also J102.11 (Pin_11), J102.8 (Pin_8)
- net EBI_A9: no longer names the net of U201.51 (PD5)
- net EBI_A9: now also J102.11 (Pin_11)
- net EBI_AD0 renamed MCU_PE7
- net EBI_AD1 renamed MCU_PE8
- net EBI_AD13: no longer names the net of U201.5 (PA4)
- net EBI_AD13: now also J102.10 (Pin_10)
- net EBI_AD14: no longer names the net of U201.6 (PA5)
- net EBI_AD14: now also J102.12 (Pin_12)
- net EBI_AD15 renamed PA6
- net PA6: now also J102.1 (Pin_1)
- net EBI_AD2 renamed MCU_PE9
- net EBI_AD3 renamed MCU_PE10
- net EBI_ALE renamed PC11
- net PC11: now also J102.11 (Pin_11)
- net EBI_ARDY: no longer names the net of J201.13 (TDO/SWO), U201.78 (PF2)
- net EBI_BL0 renamed QSPI_SCLK
- net EBI_BL1 renamed QSPI0_CS0
- net EBI_CS0 renamed QSPI0_DQ0
- net EBI_REn renamed QSPI_DQS
- net EBI_WEn renamed QSPI_CS
- new net: J102.2 (Pin_2), U201.1 (PA0)
- new net: J102.4 (Pin_4), U201.2 (PA1)
- new net: J102.6 (Pin_6), U201.3 (PA2)
- new net: J102.8 (Pin_8), U201.4 (PA3)
- no-connect marks 13 -> 10

Commit message: more pcb routing
Connections:
- net +3.3VA: no longer U201.41 (AVDD), U201.45 (AVDD)
- net GND: now also U201.41 (AVDD), U201.45 (AVDD)
- net MCU_EXTIO_PC6: now also J102.1 (Pin_1); no longer J102.6 (Pin_6)
- net MCU_EXTIO_PC7: now also J102.3 (Pin_3); no longer J102.8 (Pin_8)
- net PE0_UART0_TX: now also J102.6 (Pin_6); no longer J102.1 (Pin_1)
- net PE1_UART0_RX: now also J102.8 (Pin_8); no longer J102.3 (Pin_3)
- net PE2_UART0_CTS: now also J102.10 (Pin_10); no longer J102.5 (Pin_5)
- net PE3_UART0_RTS: now also J102.12 (Pin_12); no longer J102.7 (Pin_7)
- net PE_6: now also J102.5 (Pin_5); no longer J102.10 (Pin_10)
- net PE_7: now also J102.7 (Pin_7); no longer J102.12 (Pin_12)
- net PF10 renamed USB_D+
- net PF11 renamed USB_D-
Other:
- sheet USB3_micro_ab ports: added EFM32GG11_USB_D+, EFM32GG11_USB_D-; removed EFM32GG11_USB_DM, EFM32GG11_USB_DP
Changed lines of the file:
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@@
   (junction (at 58.674 41.91) (diameter 0) (color 0 0 0 0)
   )
-  (junction (at 77.47 63.5) (diameter 0) (color 0 0 0 0)
-  )
   (junction (at 130.81 55.88) (diameter 0) (color 0 0 0 0)
   )
@@
   (junction (at 62.23 68.58) (diameter 0) (color 0 0 0 0)
   )
-  (junction (at 77.47 60.96) (diameter 0) (color 0 0 0 0)
-  )
   (junction (at 49.276 36.83) (diameter 0) (color 0 0 0 0)
   )
@@
   (junction (at 176.53 63.5) (diameter 0) (color 0 0 0 0)
   )
+  (junction (at 82.55 63.5) (diameter 0) (color 0 0 0 0)
+  )
   (junction (at 157.48 63.5) (diameter 0) (color 0 0 0 0)
   )
@@
     (stroke (width 0) (type default))
   )
+  (wire (pts (xy 78.74 63.5) (xy 82.55 63.5))
+    (stroke (width 0) (type default))
+  )
   (wire (pts (xy 313.69 92.71) (xy 317.5 92.71))
     (stroke (width 0) (type default))
@@
     (stroke (width 0) (type default))
   )
+  (wire (pts (xy 82.55 60.96) (xy 82.55 63.5))
+    (stroke (width 0) (type default))
+  )
   (bus (pts (xy 367.03 129.54) (xy 360.68 129.54))
     (stroke (width 0) (type default))
@@
     (stroke (width 0) (type default))
   )
+  (wire (pts (xy 78.74 67.31) (xy 78.74 63.5))
+    (stroke (width 0) (type default))
+  )
   (wire (pts (xy 121.92 154.94) (xy 140.97 154.94))
     (stroke (width 0) (type default))
@@
     (stroke (width 0) (type default))
   )
-  (wire (pts (xy 77.47 60.96) (xy 82.55 60.96))
-    (stroke (width 0) (type default))
-  )
   (wire (pts (xy 20.32 41.91) (xy 30.48 41.91))
     (stroke (width 0) (type default))
@@
     (stroke (width 0) (type default))
   )
-  (wire (pts (xy 77.47 63.5) (xy 82.55 63.5))
-    (stroke (width 0) (type default))
-  )
   (wire (pts (xy 255.27 107.95) (xy 260.35 107.95))
     (stroke (width 0) (type default))
@@
     (effects (font (size 1.27 1.27)) (justify left bottom))
   )
-  (label "PF11" (at 323.85 74.93 0) (fields_autoplaced)
+  (label "USB_D-" (at 323.85 74.93 0) (fields_autoplaced)
     (effects (font (size 1.27 1.27)) (justify left bottom))
   )
@@
     (effects (font (size 1.27 1.27)) (justify right bottom))
   )
+  (label "PE3_UART0_RTS" (at 228.6 190.5 0) (fields_autoplaced)
+    (effects (font (size 1.27 1.27)) (justify left bottom))
+  )
+  (label "MCU_EXTIO_PC7" (at 201.93 180.34 180) (fields_autoplaced)
+    (effects (font (size 1.27 1.27)) (justify right bottom))
+  )
   (label "PD8" (at 283.21 138.43 0) (fields_autoplaced)
     (effects (font (size 1.27 1.27)) (justify left bottom))
@@
     (effects (font (size 1.27 1.27)) (justify left bottom))
   )
-  (label "PE1_UART0_RX" (at 201.93 180.34 180) (fields_autoplaced)
-    (effects (font (size 1.27 1.27)) (justify right bottom))
-  )
-  (label "PE2_UART0_CTS" (at 201.93 182.88 180) (fields_autoplaced)
+  (label "PE_7" (at 201.93 185.42 180) (fields_autoplaced)
     (effects (font (size 1.27 1.27)) (justify right bottom))
   )
@@
     (effects (font (size 1.27 1.27)) (justify right bottom))
   )
+  (label "PE0_UART0_TX" (at 217.17 182.88 0) (fields_autoplaced)
+    (effects (font (size 1.27 1.27)) (justify left bottom))
+  )
   (label "QSPI0_DQ1" (at 266.7 158.75 0) (fields_autoplaced)
     (effects (font (size 1.27 1.27)) (justify left bottom))
@@
     (effects (font (size 1.27 1.27)) (justify right bottom))
   )
-  (label "MCU_EXTIO_PC7" (at 217.17 185.42 0) (fields_autoplaced)
-    (effects (font (size 1.27 1.27)) (justify left bottom))
-  )
   (label "PC1" (at 283.21 143.51 0) (fields_autoplaced)
     (effects (font (size 1.27 1.27)) (justify left bottom))
@@
     (effects (font (size 1.27 1.27)) (justify right bottom))
   )
-  (label "PE_7" (at 228.6 190.5 0) (fields_autoplaced)
-    (effects (font (size 1.27 1.27)) (justify left bottom))
-  )
   (label "PC2" (at 195.58 138.43 180) (fields_autoplaced)
     (effects (font (size 1.27 1.27)) (justify right bottom))
@@
     (effects (font (size 1.27 1.27)) (justify right bottom))
   )
+  (label "MCU_EXTIO_PC6" (at 201.93 177.8 180) (fields_autoplaced)
+    (effects (font (size 1.27 1.27)) (justify right bottom))
+  )
   (label "PA8" (at 60.96 154.94 180) (fields_autoplaced)
     (effects (font (size 1.27 1.27)) (justify right bottom))
@@
     (effects (font (size 1.27 1.27)) (justify left bottom))
   )
+  (label "PE1_UART0_RX" (at 217.17 185.42 0) (fields_autoplaced)
+    (effects (font (size 1.27 1.27)) (justify left bottom))
+  )
   (label "PA9" (at 22.86 142.24 180) (fields_autoplaced)
     (effects (font (size 1.27 1.27)) (justify right bottom))
@@
     (effects (font (size 1.27 1.27)) (justify left bottom))
   )
-  (label "PF11" (at 313.69 92.71 180) (fields_autoplaced)
+  (label "USB_D+" (at 313.69 92.71 180) (fields_autoplaced)
     (effects (font (size 1.27 1.27)) (justify right bottom))
   )
@@
     (effects (font (size 1.27 1.27)) (justify right bottom))
   )
+  (label "PE_6" (at 201.93 182.88 180) (fields_autoplaced)
+    (effects (font (size 1.27 1.27)) (justify right bottom))
+  )
   (label "PE3_UART0_RTS" (at 250.19 59.69 180) (fields_autoplaced)
     (effects (font (size 1.27 1.27)) (justify right bottom))
@@
     (effects (font (size 1.27 1.27)) (justify right bottom))
   )
-  (label "PF10" (at 313.69 90.17 180) (fields_autoplaced)
+  (label "USB_D-" (at 313.69 90.17 180) (fields_autoplaced)
     (effects (font (size 1.27 1.27)) (justify right bottom))
   )
@@
     (effects (font (size 1.27 1.27)) (justify left bottom))
   )
-  (label "PF10" (at 323.85 77.47 0) (fields_autoplaced)
+  (label "USB_D+" (at 323.85 77.47 0) (fields_autoplaced)
     (effects (font (size 1.27 1.27)) (justify left bottom))
   )
@@
     (effects (font (size 1.27 1.27)) (justify right bottom))
   )
-  (label "PE3_UART0_RTS" (at 201.93 185.42 180) (fields_autoplaced)
-    (effects (font (size 1.27 1.27)) (justify right bottom))
-  )
   (label "EBI_AD6" (at 274.32 102.87 0) (fields_autoplaced)
     (effects (font (size 1.27 1.27)) (justify left bottom))
@@
     (effects (font (size 1.27 1.27)) (justify right bottom))
   )
+  (label "PE2_UART0_CTS" (at 228.6 187.96 0) (fields_autoplaced)
+    (effects (font (size 1.27 1.27)) (justify left bottom))
+  )
   (label "PC11" (at 195.58 161.29 180) (fields_autoplaced)
     (effects (font (size 1.27 1.27)) (justify right bottom))
   )
-  (label "MCU_EXTIO_PC6" (at 217.17 182.88 0) (fields_autoplaced)
-    (effects (font (size 1.27 1.27)) (justify left bottom))
-  )
   (label "PF12" (at 323.85 72.39 0) (fields_autoplaced)
     (effects (font (size 1.27 1.27)) (justify left bottom))
@@
     (effects (font (size 1.27 1.27)) (justify left bottom))
   )
-  (label "PE0_UART0_TX" (at 201.93 177.8 180) (fields_autoplaced)
-    (effects (font (size 1.27 1.27)) (justify right bottom))
-  )
   (label "PA6" (at 60.96 149.86 180) (fields_autoplaced)
     (effects (font (size 1.27 1.27)) (justify right bottom))
@@
     (effects (font (size 1.27 1.27)) (justify right bottom))
   )
-  (label "PE_6" (at 228.6 187.96 0) (fields_autoplaced)
-    (effects (font (size 1.27 1.27)) (justify left bottom))
-  )
   (label "PB12" (at 121.92 165.1 0) (fields_autoplaced)
     (effects (font (size 1.27 1.27)) (justify left bottom))
@@
     )
   )
+  (symbol (lib_id "power:GND") (at 78.74 67.31 0) (unit 1)
+    (in_bom yes) (on_board yes) (dnp no) (fields_autoplaced)
+    (property "Reference" "#PWR075" (at 78.74 73.66 0)
+      (effects (font (size 1.27 1.27)) hide)
+    )
+    (property "Value" "GND" (at 81.28 68.58 0)
+      (effects (font (size 1.27 1.27)) (justify left) hide)
+    )
+    (property "Footprint" "" (at 78.74 67.31 0)
+      (effects (font (size 1.27 1.27)) hide)
+    )
+    (property "Datasheet" "" (at 78.74 67.31 0)
+      (effects (font (size 1.27 1.27)) hide)
+    )
+    (pin "1")
+    (instances
+      (project "TripSitter"
+        (path "/5ab65702-9689-4dfd-8f10-6407062323a6/87bcf595-d251-4aa5-8b35-efc055826b19"
+          (reference "#PWR075") (unit 1)
+        )
+      )
+      (project "efm32ggxxaa"
+        (path "/86d80a6a-4f4c-4e1c-a8ce-30d9becef2f3"
+          (reference "#PWR07") (unit 1)
+        )
+      )
+      (project "RayTracingPCB"
+        (path "/e9047d94-28be-4266-894b-6ee25ef088bd/f9a74965-bde5-47a2-9f66-243cb6fc0f53"
+          (reference "#PWR07") (unit 1)
+        )
+      )
+    )
+  )
   (symbol (lib_id "Device:C_Small") (at 20.32 39.37 0) (unit 1)
     (in_bom yes) (on_board yes) (dnp no) (fields_autoplaced)
@@
       (effects (font (size 1.27 1.27)) (justify left top))
     )
-    (pin "EFM32GG11_USB_DM" output (at 317.5 90.17 180)
+    (pin "EFM32GG11_USB_D-" output (at 317.5 90.17 180)
       (effects (font (size 1.27 1.27)) (justify left))
     )
@@
       (effects (font (size 1.27 1.27)) (justify left))
     )
-    (pin "EFM32GG11_USB_DP" output (at 317.5 92.71 180)
+    (pin "EFM32GG11_USB_D+" output (at 317.5 92.71 180)
       (effects (font (size 1.27 1.27)) (justify left))
     )
