File: PCB/TripSitter/FPGA_Artix7.kicad_sch (KiCad schematic)
At the start: 31 parts, among them U1 XC7A100T-FGG484, U3 IS62WVS2568FBLL-20NLI

Commit message: pcb: re-structured PCB schematic layout (#17)
Co-authored-by: Sigvart Hovland <sigvart.m@gmail.com>
Co-authored-by: Ida-Sofie Pettersen <idasofie@Ida-Sofies-MacBook-Air.local>
Parts:
- removed C34, C88, C89: 4.7uF, Capacitor_SMD:C_0805_2012Metric_Pad1.18x1.45mm_HandSolder, symbol Device:C
- removed C87: 47uF, Capacitor_SMD:C_1210_3225Metric_Pad1.33x2.70mm_HandSolder, symbol Device:C
- removed C90, C91, C92, C93: 470nF, Capacitor_SMD:C_0201_0603Metric_Pad0.64x0.40mm_HandSolder, symbol Device:C
- added C1: 0.1uF, Capacitor_SMD:C_0603_1608Metric_Pad1.08x0.95mm_HandSolder, symbol Device:C
- added C13, C14, C15, C25, C26, C27: 470nF, Capacitor_SMD:C_0402_1005Metric_Pad0.74x0.62mm_HandSolder, symbol Device:C
- added C2, C52, C53, C54, C55, C56, C57, C58: 470nF, Capacitor_SMD:C_0201_0603Metric_Pad0.64x0.40mm_HandSolder, symbol Device:C
- added C29: 4.7uF, Capacitor_SMD:C_0402_1005Metric_Pad0.74x0.62mm_HandSolder, symbol Device:C
- added C34: 330uF, Capacitor_Tantalum_SMD:CP_EIA-7343-43_Kemet-X_Pad2.25x2.55mm_HandSolder, symbol T520V337M2R5ATE025:T520V337M2R5ATE025
- added C46, C47, C48, C49, C50: 4.7uF, Capacitor_SMD:C_0201_0603Metric_Pad0.64x0.40mm_HandSolder, symbol Device:C
- added unit 7 of U1
- added U4: DSC1001DL5-100.0000T, Footprints:CDFN4_2P5X2_MCH-L, symbol DSC1001DL5-100-0000T:DSC1001DL5-100.0000T
- C28, C31: value 470nF -> 4.7uF; footprint Capacitor_SMD:C_0201_0603Metric_Pad0.64x0.40mm_HandSolder -> Capacitor_SMD:C_0402_1005Metric_Pad0.74x0.62mm_HandSolder; Component name GRM188R71C474KA88D -> CL05A475KQ5NRNC; DK_Detail_Page https://www.digikey.no/product-detail/en/murata-electronics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 -> https://www.digikey.no/no/products/detail/samsung-electro-m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
- C30: footprint Capacitor_SMD:C_0201_0603Metric_Pad0.64x0.40mm_HandSolder -> Capacitor_SMD:C_0402_1005Metric_Pad0.74x0.62mm_HandSolder
- C32: value 470nF -> 47uF; footprint Capacitor_SMD:C_0201_0603Metric_Pad0.64x0.40mm_HandSolder -> Capacitor_SMD:C_0603_1608Metric_Pad1.08x0.95mm_HandSolder; Component name GRM188R71C474KA88D -> CL10A476MR8NZNE; DK_Detail_Page https://www.digikey.no/product-detail/en/murata-electronics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 -> https://www.digikey.no/no/products/detail/samsung-electro-m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
- C33: value 4.7uF -> 100uF; Component name C2012X7R1A475K125AC -> GRM21BR60G107ME11L; DK_Detail_Page https://www.digikey.no/product-detail/no/tdk-corporation/C2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 -> https://www.digikey.no/en/products/detail/murata-electronic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
- C35: value 47uF -> 4.7uF; footprint Capacitor_SMD:C_1210_3225Metric_Pad1.33x2.70mm_HandSolder -> Capacitor_SMD:C_0201_0603Metric_Pad0.64x0.40mm_HandSolder; Component name GRM32ER71A476ME15L -> CL03A475MQ5C65C; DK_Detail_Page https://www.digikey.no/product-detail/no/murata-electronics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 -> https://www.digikey.no/no/products/detail/samsung-electro-m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
Connections:
- net +3.3V: now also C36.1, C37.1, C38.1, C39.1, C40.1, C41.1, C42.1, C43.1, C44.1, C45.1, C80.1, C81.1, C82.1, C83.1, U1.A17 (VCCO_16), U1.B14 (VCCO_16), U1.C21 (VCCO_16), U1.D18 (VCCO_16), U1.E15 (VCCO_16), U1.F22 (VCCO_16), U1.M14 (VCCO_14), U1.P18 (VCCO_14), U1.R15 (VCCO_14), U1.T22 (VCCO_14), U1.U19 (VCCO_14), U1.Y20 (VCCO_14), C1.2, U4.1 (*STANDBY), U4.4 (VDD)
- net GND: now also C1.1, C13.2, C14.2, C15.2, C2.2, C25.2, C26.2, C27.2, C29.2, C34.1, C46.2, C47.2, C48.2, C49.2, C50.2, C52.2, C53.2, C54.2, C55.2, C56.2, C57.2, C58.2, U1.A11 (GND), U1.A12 (GND), U1.A2 (GND), U1.A22 (GND), U1.A3 (GND), U1.A5 (GND), U1.A7 (GND), U1.A9 (GND), U1.AA12 (GND), U1.AA2 (GND), U1.AA22 (GND), U1.AB19 (GND), U1.AB9 (GND), U1.B12 (GND), U1.B19 (GND), U1.B3 (GND), U1.C10 (GND), U1.C12 (GND), U1.C16 (GND), U1.C3 (GND), U1.C6 (GND), U1.D12 (GND), U1.D13 (GND), U1.D3 (GND), U1.D4 (GND), U1.D8 (GND), U1.E11 (GND), U1.E12 (VCCBATT_0), U1.E20 (GND), U1.E4 (GND), U1.E5 (GND), U1.E7 (GND), U1.E9 (GND), U1.F11 (GND), U1.F17 (GND), U1.F5 (GND), U1.G10 (GND), U1.G12 (GND), U1.G14 (GND), U1.G5 (GND), U1.G6 (GND), U1.G7 (GND), U1.G8 (GND), U1.G9 (GND), U1.H1 (GND), U1.H11 (GND), U1.H21 (GND), U1.H7 (GND), U1.H9 (GND), U1.J10 (GND), U1.J12 (GND), U1.J18 (GND), U1.J8 (GND), U1.K11 (GND), U1.K15 (GND), U1.K5 (GND), U1.K7 (GND), U1.K9 (GNDADC_0), U1.L2 (GND), U1.L22 (GND), U1.L8 (GND), U1.M11 (GND), U1.M19 (GND), U1.M7 (GND), U1.N16 (GND), U1.N6 (GND), U1.N8 (GND), U1.P11 (GND), U1.P13 (GND), U1.P3 (GND), U1.P7 (GND), U1.P9 (GND), U1.R10 (GND), U1.R12 (GND), U1.R20 (GND), U1.R8 (GND), U1.T11 (GND), U1.T17 (GND), U1.T7 (GND), U1.T9 (GND), U1.U14 (GND), U1.U4 (GND), U1.V1 (GND), U1.V11 (GND), U1.V21 (GND), U1.W18 (GND), U1.W8 (GND), U1.Y15 (GND), U1.Y5 (GND), U4.2 (GND)
- net HDMI_CEC: now also U1.B21 (IO_L21P_T3_DQS_16); no longer U1.D14 (IO_L6P_T0_16)
- net HDMI_HPD: now also U1.F19 (IO_L18P_T2_16); no longer U1.F15 (IO_0_16)
- net HDMI_SCL: now also U1.D20 (IO_L19P_T3_16); no longer U1.E16 (IO_L5P_T0_16)
- net HDMI_SDA: now also U1.F20 (IO_L18N_T2_16); no longer U1.D16 (IO_L5N_T0_16)
- net QSPI0_DQ0: now also U1.B17 (IO_L11P_T1_SRCC_16); no longer U1.W22 (IO_L7N_T1_D10_14), U1.Y16 (IO_L1P_T0_13)
- net QSPI0_DQ1: now also U1.B18 (IO_L11N_T1_SRCC_16); no longer U1.AA16 (IO_L1N_T0_13), U1.AA20 (IO_L8P_T1_D11_14)
- net QSPI0_DQ2: now also U1.A18 (IO_L17P_T2_16); no longer U1.AA21 (IO_L8N_T1_D12_14), U1.AB16 (IO_L2P_T0_13)
- net QSPI0_DQ3: now also U1.A19 (IO_L17N_T2_16); no longer U1.AB17 (IO_L2N_T0_13), U1.Y21 (IO_L9P_T1_DQS_14)
- net QSPI0_DQ4: now also U1.A16 (IO_L9N_T1_DQS_16); no longer U1.AA15 (IO_L4P_T0_13)
- net QSPI0_DQ5: now also U1.C17 (IO_L12N_T1_MRCC_16); no longer U1.AB15 (IO_L4N_T0_13)
- net QSPI0_DQ6: now also U1.A15 (IO_L9P_T1_DQS_16); no longer U1.Y13 (IO_L5P_T0_13)
- net QSPI0_DQ7: now also U1.C18 (IO_L13P_T2_MRCC_16); no longer U1.AA14 (IO_L5N_T0_13)
- net QSPI_CS: now also U1.B15 (IO_L7P_T1_16); no longer U1.Y17 (IO_0_13)
- net QSPI_DQS: now also U1.D17 (IO_L12P_T1_MRCC_16); no longer U1.AA13 (IO_L3P_T0_DQS_13)
- net QSPI_SCLK: now also U1.D14 (IO_L6P_T0_16), U3.6 (SCK); no longer U1.AB13 (IO_L3N_T0_DQS_13)
- net VGA_B1: now reaches U1.AA19 (IO_L15P_T2_DQS_RDWR_B_14)
- net VGA_B0: now reaches U1.AB20 (IO_L15N_T2_DQS_DOUT_CSO_B_14)
- net VGA_G2: now reaches U1.AB21 (IO_L10P_T1_D14_14)
- net VGA_G0: now reaches U1.AB22 (IO_L10N_T1_D15_14)
- net VGA_HSync: now reaches U1.U22 (IO_L3P_T0_DQS_PUDC_B_14)
- net VGA_VSync: now reaches U1.V22 (IO_L3N_T0_DQS_EMCCLK_14)
- net GCLK100: now reaches U1.W20 (IO_L12N_T1_MRCC_14)
- net GCLK100: now also U4.3 (OUT)
- removed net +3V3: C28.1, C30.1, C31.1, C32.1, C33.1, C35.1, C36.1, C37.1, C38.1, C39.1, C40.1, C41.1, C42.1, C43.1, C44.1, C45.1, C80.1, C81.1, C82.1, C83.1, U1.A17 (VCCO_16), U1.AA17 (VCCO_13), U1.AB14 (VCCO_13), U1.B14 (VCCO_16), U1.C21 (VCCO_16), U1.D18 (VCCO_16), U1.E15 (VCCO_16), U1.F22 (VCCO_16), U1.G19 (VCCO_15), U1.H16 (VCCO_15), U1.J13 (VCCO_15), U1.K20 (VCCO_15), U1.L17 (VCCO_15), U1.M14 (VCCO_14), U1.N21 (VCCO_15), U1.P18 (VCCO_14), U1.R15 (VCCO_14), U1.T22 (VCCO_14), U1.U19 (VCCO_14), U1.V16 (VCCO_13), U1.W13 (VCCO_13), U1.Y10 (VCCO_13), U1.Y20 (VCCO_14)
- net EBI_A0: no longer names the net of U1.J16 (IO_0_15)
- net EBI_A1: no longer names the net of U1.H13 (IO_L1P_T0_AD0P_15)
- net EBI_A10: no longer names the net of U1.H15 (IO_L5N_T0_AD9N_15)
- net EBI_A11: no longer names the net of U1.H17 (IO_L6P_T0_15)
- net EBI_A12: no longer names the net of U1.H18 (IO_L6N_T0_VREF_15)
- net EBI_A13: no longer names the net of U1.J22 (IO_L7P_T1_AD2P_15)
- net EBI_A14: no longer names the net of U1.H22 (IO_L7N_T1_AD2N_15)
- net EBI_A15: no longer names the net of U1.H20 (IO_L8P_T1_AD10P_15)
- net EBI_A16: no longer names the net of U1.G20 (IO_L8N_T1_AD10N_15)
- net EBI_A17: no longer names the net of U1.K21 (IO_L9P_T1_DQS_AD3P_15)
- net EBI_A18: no longer names the net of U1.K22 (IO_L9N_T1_DQS_AD3N_15)
- net EBI_A19: no longer names the net of U1.M21 (IO_L10P_T1_AD11P_15)
- net EBI_A2: no longer names the net of U1.G13 (IO_L1N_T0_AD0N_15)
- net EBI_A20: no longer names the net of U1.L21 (IO_L10N_T1_AD11N_15)
- net EBI_A21: no longer names the net of U1.J20 (IO_L11P_T1_SRCC_15)
- net EBI_A22: no longer names the net of U1.J21 (IO_L11N_T1_SRCC_15)
- net EBI_A23: no longer names the net of U1.J19 (IO_L12P_T1_MRCC_15)
- net EBI_A24: no longer names the net of U1.H19 (IO_L12N_T1_MRCC_15)
- net EBI_A25: no longer names the net of U1.K18 (IO_L13P_T2_MRCC_15)
- net EBI_A26: no longer names the net of U1.K19 (IO_L13N_T2_MRCC_15)
- net EBI_A27: no longer names the net of U1.L19 (IO_L14P_T2_SRCC_15)
- net EBI_A3: no longer names the net of U1.G15 (IO_L2P_T0_AD8P_15)
- net EBI_A4: no longer names the net of U1.G16 (IO_L2N_T0_AD8N_15)
- net EBI_A5: no longer names the net of U1.J14 (IO_L3P_T0_DQS_AD1P_15)
- net EBI_A6: no longer names the net of U1.H14 (IO_L3N_T0_DQS_AD1N_15)
- net EBI_A7: no longer names the net of U1.G17 (IO_L4P_T0_15)
- net EBI_A8: no longer names the net of U1.G18 (IO_L4N_T0_15)
- net EBI_A9: no longer names the net of U1.J15 (IO_L5P_T0_AD9P_15)
- net EBI_AD0: no longer names the net of U1.L20 (IO_L14N_T2_SRCC_15)
- net EBI_AD1: no longer names the net of U1.N22 (IO_L15P_T2_DQS_15)
- net EBI_AD10: no longer names the net of U1.K14 (IO_L19N_T3_A21_VREF_15)
- net EBI_AD11: no longer names the net of U1.M13 (IO_L20P_T3_A20_15)
- net EBI_AD12: no longer names the net of U1.L13 (IO_L20N_T3_A19_15)
- net EBI_AD13: no longer names the net of U1.K17 (IO_L21P_T3_DQS_15)
- net EBI_AD14: no longer names the net of U1.J17 (IO_L21N_T3_DQS_A18_15)
- net EBI_AD15: no longer names the net of U1.L14 (IO_L22P_T3_A17_15)
- net EBI_AD2: no longer names the net of U1.M22 (IO_L15N_T2_DQS_ADV_B_15)
- net EBI_AD3: no longer names the net of U1.M18 (IO_L16P_T2_A28_15)
- net EBI_AD4: no longer names the net of U1.L18 (IO_L16N_T2_A27_15)
- net EBI_AD5: no longer names the net of U1.N18 (IO_L17P_T2_A26_15)
- net EBI_AD6: no longer names the net of U1.N19 (IO_L17N_T2_A25_15)
- net EBI_AD7: no longer names the net of U1.N20 (IO_L18P_T2_A24_15)
- net EBI_AD8: no longer names the net of U1.M20 (IO_L18N_T2_A23_15)
- net EBI_AD9: no longer names the net of U1.K13 (IO_L19P_T3_A22_15)
- net EBI_ALE: no longer names the net of U1.L16 (IO_L23P_T3_FOE_B_15)
- net EBI_ARDY: no longer names the net of U1.F21 (IO_25_16)
- net EBI_BL0: no longer names the net of U1.M16 (IO_L24N_T3_RS0_15)
- net EBI_BL1: no longer names the net of U1.M17 (IO_25_15)
- net EBI_REn: no longer names the net of U1.K16 (IO_L23N_T3_FWE_B_15)
- net EBI_WEn: no longer names the net of U1.M15 (IO_L24P_T3_RS1_15)
- net HDMI_CLKN renamed MCU_PE8
- net MCU_PE8: now also U1.A14 (IO_L10N_T1_16)
- net HDMI_CLKP: no longer names the net of U1.C14 (IO_L3P_T0_DQS_16)
- net HDMI_TX0N: no longer names the net of U1.E14 (IO_L4N_T0_16)
- net HDMI_TX0P: no longer names the net of U1.E13 (IO_L4P_T0_16)
- net HDMI_TX1N: no longer names the net of U1.E17 (IO_L2N_T0_16)
- net HDMI_TX1P renamed MCU_PE9
- net HDMI_TX2N: no longer names the net of U1.F14 (IO_L1N_T0_16)
- net HDMI_TX2P: no longer names the net of U1.F13 (IO_L1P_T0_16)
- net QSPI0_CS0 renamed SRAM_QSPI0_CS0
- net SRAM_QSPI0_CS0: now also U1.C19 (IO_L13N_T2_MRCC_16); no longer U1.W21 (IO_L7P_T1_D09_14)
- net QSPI0_SCLK renamed VGA_R2
- net VGA_R2: no longer U3.6 (SCK)
- net VGA connector/VGA_B0: no longer names the net of U1.R18 (IO_L20P_T3_A08_D24_14)
- net VGA connector/VGA_B1: no longer names the net of U1.T18 (IO_L20N_T3_A07_D23_14)
- net VGA connector/VGA_B2: no longer names the net of U1.N17 (IO_L21P_T3_DQS_14)
- net VGA connector/VGA_B3: no longer names the net of U1.P17 (IO_L21N_T3_DQS_A06_D22_14)
- net VGA connector/VGA_G0: no longer names the net of U1.U17 (IO_L18P_T2_A12_D28_14)
- net VGA connector/VGA_G1: no longer names the net of U1.U18 (IO_L18N_T2_A11_D27_14)
- net VGA connector/VGA_G2: no longer names the net of U1.P14 (IO_L19P_T3_A10_D26_14)
- net VGA connector/VGA_G3: no longer names the net of U1.R14 (IO_L19N_T3_A09_D25_VREF_14)
- net VGA connector/VGA_HSync: no longer names the net of U1.P15 (IO_L22P_T3_A05_D21_14)
- net VGA connector/VGA_R0: no longer names the net of U1.V17 (IO_L16P_T2_CSI_B_14)
- net VGA connector/VGA_R1: no longer names the net of U1.W17 (IO_L16N_T2_A15_D31_14)
- net VGA connector/VGA_R2 renamed VGA_B2
- net VGA connector/VGA_R3 renamed VGA_B3
- net VGA connector/VGA_VSync: no longer names the net of U1.R16 (IO_L22N_T3_A04_D20_14)
- new net +1V0: C2.1, C27.1, C30.1, C33.1, C34.2, C35.1, C46.1, C47.1, C48.1, C49.1, C50.1, C52.1, C53.1, C54.1, C55.1, C56.1, C57.1, C58.1, U1.H10 (VCCINT), U1.H8 (VCCINT), U1.J11 (VCCBRAM), U1.J7 (VCCINT), U1.J9 (VCCINT), U1.K8 (VCCINT), U1.L11 (VCCBRAM), U1.L7 (VCCINT), U1.M8 (VCCINT), U1.N11 (VCCBRAM), U1.N7 (VCCINT), U1.P10 (VCCINT), U1.P8 (VCCINT), U1.R7 (VCCINT), U1.R9 (VCCINT), U1.T10 (VCCINT), U1.T8 (VCCINT)
- new net +1V8: C13.1, C14.1, C15.1, C25.1, C26.1, C28.1, C29.1, C31.1, C32.1, U1.H12 (VCCAUX), U1.K10 (VCCADC_0), U1.K12 (VCCAUX), U1.M12 (VCCAUX), U1.P12 (VCCAUX), U1.R11 (VCCAUX)
- new net HDMI_CLK_N: U1.G21 (IO_L24P_T3_16)
- new net HDMI_CLK_P: U1.G22 (IO_L24N_T3_16)
- new net HDMI_TX0_N: U1.E22 (IO_L22P_T3_16)
- new net HDMI_TX0_P: U1.D22 (IO_L22N_T3_16)
- new net HDMI_TX1_N: U1.C22 (IO_L20P_T3_16)
- new net HDMI_TX1_P: U1.B22 (IO_L20N_T3_16)
- new net HDMI_TX2_N: U1.A21 (IO_L21N_T3_DQS_16)
- new net HDMI_TX2_P: U1.A20 (IO_L16N_T2_16)
- new net MCU_PE7: U1.A13 (IO_L10P_T1_16)
- new net VGA_G1: U1.AA21 (IO_L8N_T1_D12_14)
- new net VGA_G3: U1.AA20 (IO_L8P_T1_D11_14)
- new net VGA_R0: U1.W22 (IO_L7N_T1_D10_14)
- new net VGA_R1: U1.W21 (IO_L7P_T1_D09_14)
- new net VGA_R3: U1.Y21 (IO_L9P_T1_DQS_14)
- now unconnected: U1.B13 (IO_L8N_T1_16), U1.B16 (IO_L7N_T1_16), U1.B20 (IO_L16P_T2_16), U1.C13 (IO_L8P_T1_16), U1.C20 (IO_L19N_T3_VREF_16), U1.D15 (IO_L6N_T0_VREF_16), U1.D19 (IO_L14N_T2_SRCC_16), U1.D21 (IO_L23N_T3_16), U1.E18 (IO_L15N_T2_DQS_16), U1.E19 (IO_L14P_T2_SRCC_16), U1.E21 (IO_L23P_T3_16), U1.F18 (IO_L15P_T2_DQS_16)
- no-connect marks 52 -> 148
Other:
- removed sheet FPGA Power Block
- note added: "Correct"
- moved on the sheet: C100, C36, C37, C38, C39, C40, C41, C42, C43, C44, C45, C80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
