File: PCB/TripSitter/MCU_usb3_microab.kicad_sch (KiCad schematic)
At the start: 9 parts, among them IC4 IP4220CZ6, J8 USB3_B_Micro

Commit message: pcb: re-structured PCB schematic layout (#17)
Co-authored-by: Sigvart Hovland <sigvart.m@gmail.com>
Co-authored-by: Ida-Sofie Pettersen <idasofie@Ida-Sofies-MacBook-Air.local>
Parts:
- removed TP2: DP_Probe, TestPoint:TestPoint_Pad_2.5x2.5mm, symbol Connector:TestPoint
- added J3: USB_B_Micro, Connector_USB:USB_Micro-B_GCT_USB3076-30-A, symbol Connector:USB_B_Micro
Connections:
- net D+: now also J3.2 (D-); no longer J8.3 (D+)
- net D-: now also J3.3 (D+); no longer J8.2 (D-), TP3.1
- net EFM32GG11_USB_ID: now also J3.4 (ID); no longer J8.4 (ID)
- net GND: now also J3.6 (Shield); no longer J8.11 (SHIELD), J8.8 (DRAIN)
- net EFM32GG11_USB_DM renamed EFM32GG11_USB_D-
- net EFM32GG11_USB_DP renamed EFM32GG11_USB_D+
- net VBUS renamed +5V
- net +5V: now also J3.1 (VBUS); no longer J8.1 (VBUS)
- no-connect marks 6 -> 2

Commit message: fix power circuit and replace jtag debug
Parts:
- removed IC4: IP4220CZ6, Package_SO:SC-74-6_1.5x2.9mm_P0.95mm, symbol IP4220CZ6:IP4220CZ6
- removed J8: USB3_B_Micro, Connector_USB:USB_Micro-B_Wuerth_629105150521_CircularHoles, symbol Connector:USB3_B_Micro
- removed TP3: DM_Probe, TestPoint:TestPoint_Pad_2.5x2.5mm, symbol Connector:TestPoint
- added IC701: IP4220CZ6, Package_SO:SC-74-6_1.5x2.9mm_P0.95mm, symbol IP4220CZ6:IP4220CZ6
Connections:
- net +5V: now also IC701.5 (VP)
- net D+: now also IC701.4 (I/O_3)
- net D-: now also IC701.6 (I/O_4)
- net EFM32GG11_USB_ID: now also IC701.1 (I/O_1)
- net GND: now also IC701.2 (GND)
