File: PCB/TripSitter/FPGA_HDMI_Connector.kicad_sch (KiCad schematic)
At the start: 16 parts, among them J4 HDMI_A_1.4, U12 TPD12S520DBT

Commit message: before
Connections:
- net +3V3 renamed +3.3V
- net HDMI_CLKN renamed HDMI_CLK_N
- net HDMI_CLKP renamed HDMI_CLK_P
- net HDMI_TX0N renamed HDMI_TX0_N
- net HDMI_TX0P renamed HDMI_TX0_P
- net HDMI_TX1N renamed HDMI_TX1_N
- net HDMI_TX1P renamed HDMI_TX1_P
- net HDMI_TX2N renamed HDMI_TX2_N
- net HDMI_TX2P renamed HDMI_TX2_P

Commit message: pcb: Finalized routing without DDR3
Added ground and power plane, layed out all the components, fanned out
BGA. QSPI between FPGA->MCU->SRAM and MCU->SRAM is routed. Most is done
but DRC does not pass so do not produce.
Parts:
- R34, R35, R36: footprint Resistor_SMD:R_0805_2012Metric_Pad1.20x1.40mm_HandSolder -> Resistor_SMD:R_0603_1608Metric_Pad0.98x0.95mm_HandSolder
Changed lines of the file:
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@@
       (effects (font (size 1.27 1.27)) (justify left))
     )
-    (property "Footprint" "Resistor_SMD:R_0805_2012Metric_Pad1.20x1.40mm_HandSolder" (at 193.802 167.64 90)
+    (property "Footprint" "Resistor_SMD:R_0603_1608Metric_Pad0.98x0.95mm_HandSolder" (at 193.802 167.64 90)
       (effects (font (size 1.27 1.27)) hide)
     )
@@
       (effects (font (size 1.27 1.27)) (justify left))
     )
-    (property "Footprint" "Resistor_SMD:R_0805_2012Metric_Pad1.20x1.40mm_HandSolder" (at 184.912 161.29 90)
+    (property "Footprint" "Resistor_SMD:R_0603_1608Metric_Pad0.98x0.95mm_HandSolder" (at 184.912 161.29 90)
       (effects (font (size 1.27 1.27)) hide)
     )
@@
       (effects (font (size 1.27 1.27)) (justify left))
     )
-    (property "Footprint" "Resistor_SMD:R_0805_2012Metric_Pad1.20x1.40mm_HandSolder" (at 168.402 156.21 90)
-      (effects (font (size 1.27 1.27)) hide)
-    )
+    (property "Footprint" "Resistor_SMD:R_0603_1608Metric_Pad0.98x0.95mm_HandSolder" (at 168.402 156.21 90)
+      (effects (font (size 1.27 1.27)) hide)
+    )

Commit message: mcu debug edit
Connections:
- net +5V: no longer D1.1 (K)
- net 5V_2: no longer names the net of R34.1, R35.1
- net 5V_2: now also D1.1 (K)
Other:
- moved on the sheet: D1
Changed lines of the file:
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@@
   (junction (at 107.95 52.07) (diameter 0) (color 0 0 0 0)
   )
+  (junction (at 143.51 90.17) (diameter 0) (color 0 0 0 0)
+  )
   (junction (at 160.02 107.95) (diameter 0) (color 0 0 0 0)
   )
@@
   )
   (no_connect (at 214.63 87.63))
-  (wire (pts (xy 256.54 142.24) (xy 261.62 142.24))
-    (stroke (width 0) (type default))
-  )
   (wire (pts (xy 250.19 196.85) (xy 257.81 196.85))
     (stroke (width 0) (type default))
@@
     (stroke (width 0) (type default))
   )
+  (wire (pts (xy 143.51 90.17) (xy 156.21 90.17))
+    (stroke (width 0) (type default))
+  )
   (wire (pts (xy 153.67 132.08) (xy 153.67 127))
     (stroke (width 0) (type default))
@@
     (stroke (width 0) (type default))
   )
-  (wire (pts (xy 245.11 142.24) (xy 248.92 142.24))
-    (stroke (width 0) (type default))
-  )
   (wire (pts (xy 222.25 100.33) (xy 224.79 100.33))
     (stroke (width 0) (type default))
@@
     (stroke (width 0) (type default))
   )
+  (wire (pts (xy 139.7 90.17) (xy 143.51 90.17))
+    (stroke (width 0) (type default))
+  )
   (wire (pts (xy 148.59 111.76) (xy 148.59 107.95))
     (stroke (width 0) (type default))
@@
     (stroke (width 0) (type default))
   )
-  (wire (pts (xy 245.11 133.35) (xy 245.11 142.24))
-    (stroke (width 0) (type default))
-  )
   (wire (pts (xy 102.87 57.15) (xy 102.87 142.24))
     (stroke (width 0) (type default))
@@
     (stroke (width 0) (type default))
   )
+  (wire (pts (xy 163.83 90.17) (xy 190.5 90.17))
+    (stroke (width 0) (type default))
+  )
   (wire (pts (xy 90.17 154.94) (xy 127 154.94))
     (stroke (width 0) (type default))
   )
+  (wire (pts (xy 143.51 85.09) (xy 143.51 90.17))
+    (stroke (width 0) (type default))
+  )
   (wire (pts (xy 204.47 82.55) (xy 214.63 82.55))
     (stroke (width 0) (type default))
@@
     (stroke (width 0) (type default))
   )
-  (wire (pts (xy 139.7 125.73) (xy 139.7 128.27))
+  (wire (pts (xy 139.7 90.17) (xy 139.7 128.27))
     (stroke (width 0) (type default))
   )
@@
     (stroke (width 0) (type default))
   )
-  (wire (pts (xy 190.5 152.4) (xy 190.5 154.94))
+  (wire (pts (xy 190.5 90.17) (xy 190.5 154.94))
     (stroke (width 0) (type default))
   )
   (wire (pts (xy 107.95 52.07) (xy 107.95 137.16))
     (stroke (width 0) (type default))
-  )
-  (label "5V_1" (at 245.11 142.24 0) (fields_autoplaced)
-    (effects (font (size 1.27 1.27)) (justify left bottom))
   )
   (label "5V2" (at 254 39.37 0) (fields_autoplaced)
     (effects (font (size 1.27 1.27)) (justify left bottom))
   )
-  (label "5V_1" (at 139.7 125.73 0) (fields_autoplaced)
-    (effects (font (size 1.27 1.27)) (justify left bottom))
-  )
-  (label "5V2" (at 261.62 142.24 0) (fields_autoplaced)
-    (effects (font (size 1.27 1.27)) (justify left bottom))
-  )
   (label "CEC" (at 207.01 74.93 0) (fields_autoplaced)
-    (effects (font (size 1.27 1.27)) (justify left bottom))
-  )
-  (label "5V_2" (at 190.5 152.4 0) (fields_autoplaced)
     (effects (font (size 1.27 1.27)) (justify left bottom))
   )
@@
     )
   )
-  (symbol (lib_id "Device:D") (at 252.73 142.24 180) (unit 1)
+  (symbol (lib_id "Device:D") (at 160.02 90.17 180) (unit 1)
     (in_bom yes) (on_board yes) (dnp no) (fields_autoplaced)
-    (property "Reference" "D1" (at 252.73 135.89 0)
-      (effects (font (size 1.27 1.27)))
-    )
-    (property "Value" "D" (at 252.73 138.43 0)
-      (effects (font (size 1.27 1.27)))
-    )
-    (property "Footprint" "Diode_SMD:D_0201_0603Metric_Pad0.64x0.40mm_HandSolder" (at 252.73 142.24 0)
-      (effects (font (size 1.27 1.27)) hide)
-    )
-    (property "Datasheet" "~" (at 252.73 142.24 0)
-      (effects (font (size 1.27 1.27)) hide)
-    )
-    (property "Sim.Device" "D" (at 252.73 142.24 0)
-      (effects (font (size 1.27 1.27)) hide)
-    )
-    (property "Sim.Pins" "1=K 2=A" (at 252.73 142.24 0)
+    (property "Reference" "D1" (at 160.02 83.82 0)
+      (effects (font (size 1.27 1.27)))
+    )
+    (property "Value" "D" (at 160.02 86.36 0)
+      (effects (font (size 1.27 1.27)))
+    )
+    (property "Footprint" "Diode_SMD:D_0201_0603Metric_Pad0.64x0.40mm_HandSolder" (at 160.02 90.17 0)
+      (effects (font (size 1.27 1.27)) hide)
+    )
+    (property "Datasheet" "~" (at 160.02 90.17 0)
+      (effects (font (size 1.27 1.27)) hide)
+    )
+    (property "Sim.Device" "D" (at 160.02 90.17 0)
+      (effects (font (size 1.27 1.27)) hide)
+    )
+    (property "Sim.Pins" "1=K 2=A" (at 160.02 90.17 0)
       (effects (font (size 1.27 1.27)) hide)
     )
@@
         (path "/e9047d94-28be-4266-894b-6ee25ef088bd/81518b75-edd1-4c8b-a158-389aac8d5196"
           (reference "D1") (unit 1)
+        )
+      )
+    )
+  )
+  (symbol (lib_id "power:+5V") (at 143.51 85.09 0) (unit 1)
+    (in_bom yes) (on_board yes) (dnp no) (fields_autoplaced)
+    (property "Reference" "#PWR016" (at 143.51 88.9 0)
+      (effects (font (size 1.27 1.27)) hide)
+    )
+    (property "Value" "+5V" (at 143.51 80.01 0)
+      (effects (font (size 1.27 1.27)))
+    )
+    (property "Footprint" "" (at 143.51 85.09 0)
+      (effects (font (size 1.27 1.27)) hide)
+    )
+    (property "Datasheet" "" (at 143.51 85.09 0)
+      (effects (font (size 1.27 1.27)) hide)
+    )
+    (pin "1")
+    (instances
+      (project "TripSitter"
+        (path "/5ab65702-9689-4dfd-8f10-6407062323a6/095fe883-dc50-4e06-a886-995eeb7c2300/ae3612c6-9651-4a37-8de7-7277774520fa"
+          (reference "#PWR016") (unit 1)
         )
       )
@@
         )
       )
-    )
-  )
-  (symbol (lib_id "power:+5V") (at 245.11 133.35 0) (unit 1)
-    (in_bom yes) (on_board yes) (dnp no) (fields_autoplaced)
-    (property "Reference" "#PWR05" (at 245.11 137.16 0)
-      (effects (font (size 1.27 1.27)) hide)
-    )
-    (property "Value" "+5V" (at 245.11 128.27 0)
-      (effects (font (size 1.27 1.27)))
-    )
-    (property "Footprint" "" (at 245.11 133.35 0)
-      (effects (font (size 1.27 1.27)) hide)
-    )
-    (property "Datasheet" "" (at 245.11 133.35 0)
-      (effects (font (size 1.27 1.27)) hide)
-    )
-    (pin "1")
-    (instances
-      (project "hdmi_connector"
-        (path "/402b0016-56b9-4470-870c-5895a0afd1d9"
-          (reference "#PWR05") (unit 1)
-        )
-      )
-      (project "TripSitter"
-        (path "/5ab65702-9689-4dfd-8f10-6407062323a6/095fe883-dc50-4e06-a886-995eeb7c2300/ae3612c6-9651-4a37-8de7-7277774520fa"
-          (reference "#PWR069") (unit 1)
-        )
-      )
-      (project "RayTracingPCB"
-        (path "/e9047d94-28be-4266-894b-6ee25ef088bd/81518b75-edd1-4c8b-a158-389aac8d5196"
-          (reference "#PWR05") (unit 1)
-        )
-      )
