File: PCB/TripSitter/TripSitter.kicad_pcb (KiCad board)
At the start: 6 copper layers, 177 parts, among them IC1 MT25QL256ABA1EW9-0SIT, IC2 MT41J128M16JT-125_K, IC4 IP4220CZ6, J1 Conn_ARM_JTAG_SWD_20, J2 DE15_Plug_HighDensity_Mountin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, J3 Conn_ARM_JTAG_SWD_20, J4 USB_B_Micro, J5 Jack-DC, J6 EFM32_PinHeader_PortE, J7 HDMI_A_1.4, J8 USB3_B_Micro, SW1 SW_Push_Open, SW2 SW_DPDT_x2, SW3 SW_DIP_x05, U1 XC7A100T-FGG484, U2 TPS54325_PWP_14, U3 IS62WVS2568FBLL-20NLI, U4 EFM32GG11B420F2048GQ100, U5 TPS54294PWP, U6 IS62WVS2568FBLL-20NLI, U7 TPD12S520DBT, X1 XO53 100Mhz, Y1 48MHz

Commit message: attempt at routing
Parts:
- IC2: footprint footprints:FBGA96_8X14_MRN -> Package_BGA:Micron_FBGA-96_8x14mm_Layout9x16_P0.8mm; moved to B.Cu
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Connections:
- net /FPGA Artix-7 100T 1FGG484C/DDR3/DDR3_LDQS renamed /FPGA Artix-7 100T 1FGG484C/DDR3/DDR3_LDQS_P
- net /FPGA Artix-7 100T 1FGG484C/DDR3/DDR3_nLDQS renamed /FPGA Artix-7 100T 1FGG484C/DDR3/DDR3_LDQS_N
- IC2 pad B7: /FPGA Artix-7 100T 1FGG484C/DDR3/DDR3_nUDQS -> /FPGA Artix-7 100T 1FGG484C/DDR3/DDR3_UDQS_N
- IC2 pad C7: /FPGA Artix-7 100T 1FGG484C/DDR3/DDR3_UDQS -> /FPGA Artix-7 100T 1FGG484C/DDR3/DDR3_UDQS_P
- IC2 pad J7: /FPGA Artix-7 100T 1FGG484C/DDR3/DDR3_CK -> /FPGA Artix-7 100T 1FGG484C/DDR3/DDR3_CK_P
- IC2 pad K7: /FPGA Artix-7 100T 1FGG484C/DDR3/DDR3_nCK -> /FPGA Artix-7 100T 1FGG484C/DDR3/DDR3_CK_N
- U1 pad A1: unconnected-(U1C-IO_25_35-PadL6) -> (no net)
- U1 pad A10: unconnected-(U1D-MGTPRXN0_216-PadA8) -> unconnected-(U1D-MGTPRXN2_216-PadA10)
- U1 pad A13: unconnected-(U1B-IO_L10N_T1_16-PadA14) -> unconnected-(U1B-IO_L10P_T1_16-PadA13)
- U1 pad A15: unconnected-(U1B-IO_L10N_T1_16-PadA14) -> unconnected-(U1B-IO_L9P_T1_DQS_16-PadA15)
- U1 pad A16: unconnected-(U1B-IO_L10N_T1_16-PadA14) -> unconnected-(U1B-IO_L9N_T1_DQS_16-PadA16)
- U1 pad A18: unconnected-(U1B-IO_L10N_T1_16-PadA14) -> unconnected-(U1B-IO_L17P_T2_16-PadA18)
- U1 pad A19: unconnected-(U1B-IO_L10N_T1_16-PadA14) -> unconnected-(U1B-IO_L17N_T2_16-PadA19)
- U1 pad A20: unconnected-(U1B-IO_L10N_T1_16-PadA14) -> unconnected-(U1B-IO_L16N_T2_16-PadA20)
- U1 pad A21: unconnected-(U1B-IO_L10N_T1_16-PadA14) -> unconnected-(U1B-IO_L21N_T3_DQS_16-PadA21)
- U1 pad A4: unconnected-(U1D-MGTPRXN0_216-PadA8) -> unconnected-(U1D-MGTPTXN0_216-PadA4)
- U1 pad A6: unconnected-(U1D-MGTPRXN0_216-PadA8) -> unconnected-(U1D-MGTPTXN2_216-PadA6)
- U1 pad AA1: /FPGA Artix-7 100T 1FGG484C/DDR3/DDR3_UDM -> /FPGA Artix-7 100T 1FGG484C/DDR3/DDR3_nRESET
- U1 pad AA3: /FPGA Artix-7 100T 1FGG484C/DDR3/DDR3_nUDQS -> /FPGA Artix-7 100T 1FGG484C/DDR3/DDR3_UDQS_P
- U1 pad AA4: /FPGA Artix-7 100T 1FGG484C/DDR3/DDR3_DQ13 -> /FPGA Artix-7 100T 1FGG484C/DDR3/DDR3_BA2
- U1 pad AA5: /FPGA Artix-7 100T 1FGG484C/DDR3/DDR3_DQ11 -> /FPGA Artix-7 100T 1FGG484C/DDR3/DDR3_DQ14
- U1 pad AA6: /FPGA Artix-7 100T 1FGG484C/DDR3/DDR3_A9 -> /FPGA Artix-7 100T 1FGG484C/DDR3/DDR3_A12
- U1 pad AA8: /FPGA Artix-7 100T 1FGG484C/DDR3/DDR3_A7 -> /FPGA Artix-7 100T 1FGG484C/DDR3/DDR3_A6
- U1 pad AB1: /FPGA Artix-7 100T 1FGG484C/DDR3/DDR3_DQ12 -> /FPGA Artix-7 100T 1FGG484C/DDR3/DDR3_A13
- U1 pad AB2: /FPGA Artix-7 100T 1FGG484C/DDR3/DDR3_DQ14 -> /FPGA Artix-7 100T 1FGG484C/DDR3/DDR3_A9
- U1 pad AB3: /FPGA Artix-7 100T 1FGG484C/DDR3/DDR3_DQ10 -> /FPGA Artix-7 100T 1FGG484C/DDR3/DDR3_A2
- U1 pad AB5: /FPGA Artix-7 100T 1FGG484C/DDR3/DDR3_DQ8 -> /FPGA Artix-7 100T 1FGG484C/DDR3/DDR3_A0
- U1 pad AB6: /FPGA Artix-7 100T 1FGG484C/DDR3/DDR3_A6 -> /FPGA Artix-7 100T 1FGG484C/DDR3/DDR3_A10
- U1 pad AB7: /FPGA Artix-7 100T 1FGG484C/DDR3/DDR3_ODT -> /FPGA Artix-7 100T 1FGG484C/DDR3/DDR3_A11
- U1 pad AB8: /FPGA Artix-7 100T 1FGG484C/DDR3/DDR3_A11 -> /FPGA Artix-7 100T 1FGG484C/DDR3/DDR3_A8
- U1 pad B1: unconnected-(U1C-IO_25_35-PadL6) -> (no net)
- U1 pad B10: unconnected-(U1D-MGTPRXN0_216-PadA8) -> unconnected-(U1D-MGTPRXP2_216-PadB10)
- U1 pad B11: unconnected-(U1D-MGTPRXN0_216-PadA8) -> unconnected-(U1E-MGTAVTT-PadB11)
- U1 pad B13: unconnected-(U1B-IO_L10N_T1_16-PadA14) -> unconnected-(U1B-IO_L8N_T1_16-PadB13)
- U1 pad B15: unconnected-(U1B-IO_L10N_T1_16-PadA14) -> unconnected-(U1B-IO_L7P_T1_16-PadB15)
- U1 pad B16: unconnected-(U1B-IO_L10N_T1_16-PadA14) -> unconnected-(U1B-IO_L7N_T1_16-PadB16)
- U1 pad B17: unconnected-(U1B-IO_L10N_T1_16-PadA14) -> unconnected-(U1B-IO_L11P_T1_SRCC_16-PadB17)
- U1 pad B18: unconnected-(U1B-IO_L10N_T1_16-PadA14) -> unconnected-(U1B-IO_L11N_T1_SRCC_16-PadB18)
- U1 pad B2: unconnected-(U1C-IO_25_35-PadL6) -> (no net)
- U1 pad B20: unconnected-(U1B-IO_L10N_T1_16-PadA14) -> unconnected-(U1B-IO_L16P_T2_16-PadB20)
- U1 pad B21: unconnected-(U1B-IO_L10N_T1_16-PadA14) -> unconnected-(U1B-IO_L21P_T3_DQS_16-PadB21)
- U1 pad B22: unconnected-(U1B-IO_L10N_T1_16-PadA14) -> unconnected-(U1B-IO_L20N_T3_16-PadB22)
- U1 pad B4: unconnected-(U1D-MGTPRXN0_216-PadA8) -> unconnected-(U1D-MGTPTXP0_216-PadB4)
- U1 pad B5: unconnected-(U1D-MGTPRXN0_216-PadA8) -> unconnected-(U1E-MGTAVTT-PadB5)
- U1 pad B6: unconnected-(U1D-MGTPRXN0_216-PadA8) -> unconnected-(U1D-MGTPTXP2_216-PadB6)
- U1 pad B7: unconnected-(U1D-MGTPRXN0_216-PadA8) -> unconnected-(U1E-MGTAVTT-PadB7)
- U1 pad B8: unconnected-(U1D-MGTPRXN0_216-PadA8) -> unconnected-(U1D-MGTPRXP0_216-PadB8)
- U1 pad B9: unconnected-(U1D-MGTPRXN0_216-PadA8) -> unconnected-(U1E-MGTAVTT-PadB9)
- U1 pad C1: +1V5 -> (no net)
- U1 pad C11: unconnected-(U1D-MGTPRXN0_216-PadA8) -> unconnected-(U1D-MGTPRXN1_216-PadC11)
- U1 pad C13: unconnected-(U1B-IO_L10N_T1_16-PadA14) -> unconnected-(U1B-IO_L8P_T1_16-PadC13)
- U1 pad C17: unconnected-(U1B-IO_L10N_T1_16-PadA14) -> unconnected-(U1B-IO_L12N_T1_MRCC_16-PadC17)
- U1 pad C18: unconnected-(U1B-IO_L10N_T1_16-PadA14) -> unconnected-(U1B-IO_L13P_T2_MRCC_16-PadC18)
- U1 pad C19: unconnected-(U1B-IO_L10N_T1_16-PadA14) -> unconnected-(U1B-IO_L13N_T2_MRCC_16-PadC19)
- U1 pad C2: unconnected-(U1C-IO_25_35-PadL6) -> (no net)
- U1 pad C20: unconnected-(U1B-IO_L10N_T1_16-PadA14) -> unconnected-(U1B-IO_L19N_T3_VREF_16-PadC20)
- U1 pad C22: unconnected-(U1B-IO_L10N_T1_16-PadA14) -> unconnected-(U1B-IO_L20P_T3_16-PadC22)
- U1 pad C4: unconnected-(U1D-MGTPRXN0_216-PadA8) -> unconnected-(U1E-MGTAVTT-PadC4)
- U1 pad C5: unconnected-(U1D-MGTPRXN0_216-PadA8) -> unconnected-(U1D-MGTPTXN1_216-PadC5)
- U1 pad C7: unconnected-(U1D-MGTPRXN0_216-PadA8) -> unconnected-(U1D-MGTPTXN3_216-PadC7)
- U1 pad C8: unconnected-(U1D-MGTPRXN0_216-PadA8) -> unconnected-(U1E-MGTAVTT-PadC8)
- U1 pad C9: unconnected-(U1D-MGTPRXN0_216-PadA8) -> unconnected-(U1D-MGTPRXN3_216-PadC9)
- U1 pad D1: unconnected-(U1C-IO_25_35-PadL6) -> (no net)
- U1 pad D10: unconnected-(U1D-MGTPRXN0_216-PadA8) -> unconnected-(U1E-MGTAVCC-PadD10)
- U1 pad D11: unconnected-(U1D-MGTPRXN0_216-PadA8) -> unconnected-(U1D-MGTPRXP1_216-PadD11)
- U1 pad D15: unconnected-(U1B-IO_L10N_T1_16-PadA14) -> unconnected-(U1B-IO_L6N_T0_VREF_16-PadD15)
- U1 pad D17: unconnected-(U1B-IO_L10N_T1_16-PadA14) -> unconnected-(U1B-IO_L12P_T1_MRCC_16-PadD17)
- U1 pad D19: unconnected-(U1B-IO_L10N_T1_16-PadA14) -> unconnected-(U1B-IO_L14N_T2_SRCC_16-PadD19)
- U1 pad D2: unconnected-(U1C-IO_25_35-PadL6) -> (no net)
- U1 pad D20: unconnected-(U1B-IO_L10N_T1_16-PadA14) -> unconnected-(U1B-IO_L19P_T3_16-PadD20)
- U1 pad D21: unconnected-(U1B-IO_L10N_T1_16-PadA14) -> unconnected-(U1B-IO_L23N_T3_16-PadD21)
- U1 pad D22: unconnected-(U1B-IO_L10N_T1_16-PadA14) -> unconnected-(U1B-IO_L22N_T3_16-PadD22)
- U1 pad D5: unconnected-(U1D-MGTPRXN0_216-PadA8) -> unconnected-(U1D-MGTPTXP1_216-PadD5)
- U1 pad D6: unconnected-(U1D-MGTPRXN0_216-PadA8) -> unconnected-(U1E-MGTAVCC-PadD6)
- U1 pad D7: unconnected-(U1D-MGTPRXN0_216-PadA8) -> unconnected-(U1D-MGTPTXP3_216-PadD7)
- U1 pad D9: unconnected-(U1D-MGTPRXN0_216-PadA8) -> unconnected-(U1D-MGTPRXP3_216-PadD9)
- U1 pad E1: unconnected-(U1C-IO_25_35-PadL6) -> (no net)
- U1 pad E10: unconnected-(U1D-MGTPRXN0_216-PadA8) -> unconnected-(U1D-MGTREFCLK1N_216-PadE10)
- U1 pad E18: unconnected-(U1B-IO_L10N_T1_16-PadA14) -> unconnected-(U1B-IO_L15N_T2_DQS_16-PadE18)
- U1 pad E19: unconnected-(U1B-IO_L10N_T1_16-PadA14) -> unconnected-(U1B-IO_L14P_T2_SRCC_16-PadE19)
- U1 pad E2: unconnected-(U1C-IO_25_35-PadL6) -> (no net)
- U1 pad E21: unconnected-(U1B-IO_L10N_T1_16-PadA14) -> unconnected-(U1B-IO_L23P_T3_16-PadE21)
- U1 pad E22: unconnected-(U1B-IO_L10N_T1_16-PadA14) -> unconnected-(U1B-IO_L22P_T3_16-PadE22)
- U1 pad E3: unconnected-(U1C-IO_25_35-PadL6) -> (no net)
- U1 pad E6: unconnected-(U1D-MGTPRXN0_216-PadA8) -> unconnected-(U1D-MGTREFCLK0N_216-PadE6)
- U1 pad E8: unconnected-(U1D-MGTPRXN0_216-PadA8) -> unconnected-(U1E-MGTAVCC-PadE8)
- U1 pad F1: unconnected-(U1C-IO_25_35-PadL6) -> (no net)
- U1 pad F10: unconnected-(U1D-MGTPRXN0_216-PadA8) -> unconnected-(U1D-MGTREFCLK1P_216-PadF10)
- U1 pad F18: unconnected-(U1B-IO_L10N_T1_16-PadA14) -> unconnected-(U1B-IO_L15P_T2_DQS_16-PadF18)
- U1 pad F19: unconnected-(U1B-IO_L10N_T1_16-PadA14) -> unconnected-(U1B-IO_L18P_T2_16-PadF19)
- U1 pad F2: +1V5 -> (no net)
- U1 pad F20: unconnected-(U1B-IO_L10N_T1_16-PadA14) -> unconnected-(U1B-IO_L18N_T2_16-PadF20)
- U1 pad F3: unconnected-(U1C-IO_25_35-PadL6) -> (no net)
- U1 pad F4: /FPGA Artix-7 100T 1FGG484C/DDR3/XO_Enable -> (no net)
- U1 pad F6: unconnected-(U1D-MGTPRXN0_216-PadA8) -> unconnected-(U1D-MGTREFCLK0P_216-PadF6)
- U1 pad F7: unconnected-(U1D-MGTPRXN0_216-PadA8) -> unconnected-(U1E-MGTAVCC-PadF7)
- U1 pad F8: unconnected-(U1D-MGTPRXN0_216-PadA8) -> unconnected-(U1E-MGTRREF_216-PadF8)
- U1 pad F9: unconnected-(U1D-MGTPRXN0_216-PadA8) -> unconnected-(U1E-MGTAVCC-PadF9)
- U1 pad G1: unconnected-(U1C-IO_25_35-PadL6) -> (no net)
- U1 pad G2: unconnected-(U1C-IO_25_35-PadL6) -> (no net)
- U1 pad G21: unconnected-(U1B-IO_L10N_T1_16-PadA14) -> unconnected-(U1B-IO_L24P_T3_16-PadG21)
- U1 pad G22: unconnected-(U1B-IO_L10N_T1_16-PadA14) -> unconnected-(U1B-IO_L24N_T3_16-PadG22)
- U1 pad G3: unconnected-(U1C-IO_25_35-PadL6) -> (no net)
- U1 pad G4: unconnected-(U1C-IO_25_35-PadL6) -> (no net)
- U1 pad H2: unconnected-(U1C-IO_25_35-PadL6) -> (no net)
- U1 pad H3: unconnected-(U1C-IO_25_35-PadL6) -> (no net)
- U1 pad H4: unconnected-(U1C-IO_25_35-PadL6) -> (no net)
- U1 pad H5: unconnected-(U1C-IO_25_35-PadL6) -> (no net)
- U1 pad H6: +1V5 -> (no net)
- U1 pad J1: unconnected-(U1C-IO_25_35-PadL6) -> (no net)
- U1 pad J2: unconnected-(U1C-IO_25_35-PadL6) -> (no net)
- U1 pad J3: +1V5 -> (no net)
- U1 pad J4: unconnected-(U1C-IO_25_35-PadL6) -> (no net)
- U1 pad J5: unconnected-(U1C-IO_25_35-PadL6) -> (no net)
- U1 pad J6: unconnected-(U1C-IO_25_35-PadL6) -> (no net)
- U1 pad K1: unconnected-(U1C-IO_25_35-PadL6) -> (no net)
- U1 pad K2: unconnected-(U1C-IO_25_35-PadL6) -> (no net)
- U1 pad K3: unconnected-(U1C-IO_25_35-PadL6) -> (no net)
- U1 pad K4: unconnected-(U1C-IO_25_35-PadL6) -> (no net)
- U1 pad K6: unconnected-(U1C-IO_25_35-PadL6) -> (no net)
- U1 pad L1: unconnected-(U1C-IO_25_35-PadL6) -> (no net)
- U1 pad L3: unconnected-(U1C-IO_25_35-PadL6) -> (no net)
- U1 pad L4: unconnected-(U1C-IO_25_35-PadL6) -> (no net)
- U1 pad L5: unconnected-(U1C-IO_25_35-PadL6) -> (no net)
- U1 pad L6: unconnected-(U1C-IO_25_35-PadL6) -> (no net)
- U1 pad M1: unconnected-(U1C-IO_25_35-PadL6) -> (no net)
- U1 pad M2: unconnected-(U1C-IO_25_35-PadL6) -> (no net)
- U1 pad M3: unconnected-(U1C-IO_25_35-PadL6) -> (no net)
- U1 pad M4: +1V5 -> (no net)
- U1 pad M5: unconnected-(U1C-IO_25_35-PadL6) -> (no net)
- U1 pad M6: unconnected-(U1C-IO_25_35-PadL6) -> (no net)
- U1 pad N1: +1V5 -> (no net)
- U1 pad N2: unconnected-(U1C-IO_25_35-PadL6) -> (no net)
- U1 pad N3: unconnected-(U1C-IO_25_35-PadL6) -> (no net)
- U1 pad N4: unconnected-(U1C-IO_25_35-PadL6) -> (no net)
- U1 pad N5: unconnected-(U1C-IO_25_35-PadL6) -> (no net)
- U1 pad P1: unconnected-(U1C-IO_25_35-PadL6) -> (no net)
- U1 pad P2: unconnected-(U1C-IO_25_35-PadL6) -> (no net)
- U1 pad P4: unconnected-(U1C-IO_25_35-PadL6) -> (no net)
- U1 pad P5: unconnected-(U1C-IO_25_35-PadL6) -> (no net)
- U1 pad P6: unconnected-(U1C-IO_25_35-PadL6) -> (no net)
- U1 pad R1: unconnected-(U1C-IO_25_35-PadL6) -> (no net)
- U1 pad R6: /FPGA Artix-7 100T 1FGG484C/DDR3/DDR3_BA0 -> /FPGA Artix-7 100T 1FGG484C/DDR3/DDR3_UDM
- U1 pad T1: /FPGA Artix-7 100T 1FGG484C/DDR3/DDR3_LDM -> /FPGA Artix-7 100T 1FGG484C/DDR3/DDR3_BA0
- U1 pad T3: /FPGA Artix-7 100T 1FGG484C/DDR3/DDR3_nRESET -> /FPGA Artix-7 100T 1FGG484C/DDR3/DDR3_DQ6
- U1 pad T5: /FPGA Artix-7 100T 1FGG484C/DDR3/DDR3_BA1 -> /FPGA Artix-7 100T 1FGG484C/DDR3/DDR3_DQ11
- U1 pad T6: /FPGA Artix-7 100T 1FGG484C/DDR3/DDR3_A1 -> /FPGA Artix-7 100T 1FGG484C/DDR3/DDR3_ODT
- U1 pad U1: /FPGA Artix-7 100T 1FGG484C/DDR3/DDR3_DQ5 -> /FPGA Artix-7 100T 1FGG484C/DDR3/DDR3_A3
- U1 pad V3: /FPGA Artix-7 100T 1FGG484C/DDR3/DDR3_A14 -> /FPGA Artix-7 100T 1FGG484C/DDR3/XO_Enable
- U1 pad V5: /FPGA Artix-7 100T 1FGG484C/DDR3/DDR3_A2 -> /FPGA Artix-7 100T 1FGG484C/DDR3/DDR3_DQ10
- U1 pad V7: /FPGA Artix-7 100T 1FGG484C/DDR3/DDR3_A3 -> /FPGA Artix-7 100T 1FGG484C/DDR3/DDR3_DQ5
- U1 pad V8: /FPGA Artix-7 100T 1FGG484C/DDR3/DDR3_nCK -> /FPGA Artix-7 100T 1FGG484C/DDR3/DDR3_CK_P
- U1 pad V9: /FPGA Artix-7 100T 1FGG484C/DDR3/DDR3_CK -> /FPGA Artix-7 100T 1FGG484C/DDR3/DDR3_CK_N
- U1 pad W1: /FPGA Artix-7 100T 1FGG484C/DDR3/DDR3_DQ0 -> /FPGA Artix-7 100T 1FGG484C/DDR3/DDR3_A5
- U1 pad W5: /FPGA Artix-7 100T 1FGG484C/DDR3/DDR3_A0 -> /FPGA Artix-7 100T 1FGG484C/DDR3/DDR3_DQ8
- U1 pad W6: /FPGA Artix-7 100T 1FGG484C/DDR3/DDR3_BA2 -> /FPGA Artix-7 100T 1FGG484C/DDR3/DDR3_DQ12
- U1 pad W7: /FPGA Artix-7 100T 1FGG484C/DDR3/DDR3_A4 -> /FPGA Artix-7 100T 1FGG484C/DDR3/DDR3_DQ13
- U1 pad W9: /FPGA Artix-7 100T 1FGG484C/DDR3/DDR3_A8 -> /FPGA Artix-7 100T 1FGG484C/DDR3/DDR3_BA1
- U1 pad Y1: /FPGA Artix-7 100T 1FGG484C/DDR3/DDR3_DQ6 -> /FPGA Artix-7 100T 1FGG484C/DDR3/DDR3_A7
- U1 pad Y3: /FPGA Artix-7 100T 1FGG484C/DDR3/DDR3_UDQS -> /FPGA Artix-7 100T 1FGG484C/DDR3/DDR3_UDQS_N
- U1 pad Y6: /FPGA Artix-7 100T 1FGG484C/DDR3/DDR3_A10 -> /FPGA Artix-7 100T 1FGG484C/DDR3/DDR3_A1
- U1 pad Y7: /FPGA Artix-7 100T 1FGG484C/DDR3/DDR3_A12 -> /FPGA Artix-7 100T 1FGG484C/DDR3/DDR3_LDM
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Routing:
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
Commit message: before
Parts:
- removed C48: 1uF, Capacitor_SMD:C_0201_0603Metric_Pad0.64x0.40mm_HandSolder
- removed C50, C58, C63: 10uF, Capacitor_SMD:C_0402_1005Metric_Pad0.74x0.62mm_HandSolder
- removed C51, C97: 0.1uF, Capacitor_SMD:C_0201_0603Metric_Pad0.64x0.40mm_HandSolder
- removed C56: 10nF, Capacitor_SMD:C_0402_1005Metric_Pad0.74x0.62mm_HandSolder
- removed C61: 100uF, Capacitor_SMD:C_1210_3225Metric_Pad1.33x2.70mm_HandSolder
- removed C99: 100uF, Capacitor_SMD:C_0805_2012Metric_Pad1.18x1.45mm_HandSolder
- removed IC4: IP4220CZ6, Package_SO:SC-74-6_1.5x2.9mm_P0.95mm
- removed J3: Conn_ARM_JTAG_SWD_20, Connector_PinHeader_1.00mm:PinHeader_2x10_P1.00mm_Vertical
- removed J4: USB_B_Micro, Connector_USB:USB_Micro-B_Wuerth_629105150521_CircularHoles
- removed J5: Jack-DC, Connector_BarrelJack:BarrelJack_CUI_PJ-063AH_Horizontal_CircularHoles
- removed J8: USB3_B_Micro, Connector_USB:USB_Micro-B_Wuerth_629105150521_CircularHoles
- removed L1, L2: 1.5uH, Inductor_SMD:L_0805_2012Metric_Pad1.15x1.40mm_HandSolder
- removed the R19 at (62.9, 79.8)
- removed R24: 100k, Resistor_SMD:R_0805_2012Metric_Pad1.20x1.40mm_HandSolder
- removed SW2: SW_DPDT_x2, Button_Switch_SMD:SW_DPDT_CK_JS202011JCQN
- removed SW3: SW_DIP_x05, Connector_PinHeader_1.27mm:PinHeader_2x05_P1.27mm_Vertical
- removed TP2: DP_Probe, TestPoint:TestPoint_Pad_2.5x2.5mm
- removed TP3: DM_Probe, TestPoint:TestPoint_Pad_2.5x2.5mm
- removed U3: IS62WVS2568FBLL-20NLI, Package_SO:SOIC-8_3.9x4.9mm_P1.27mm
- removed U4: EFM32GG11B420F2048GQ100, Package_QFP:TQFP-100_14x14mm_P0.5mm
- removed Y1: 48MHz, Crystal:Crystal_SMD_2016-4Pin_2.0x1.6mm
- added C11: 470nF, Capacitor_SMD:C_0201_0603Metric_Pad0.64x0.40mm_HandSolder, F.Cu at (13.7, 27.0)
- added C12: 4.7uF, Capacitor_SMD:C_0805_2012Metric_Pad1.18x1.45mm_HandSolder, F.Cu at (14.7, 22.9)
- added C13: 4.7uF, Capacitor_SMD:C_0805_2012Metric_Pad1.18x1.45mm_HandSolder, F.Cu at (7.92, 22.9)
- added C14: 4.7uF, Capacitor_SMD:C_0805_2012Metric_Pad1.18x1.45mm_HandSolder, F.Cu at (7.92, 25.9)
- added C15: 47uF, Capacitor_SMD:C_1210_3225Metric_Pad1.33x2.70mm_HandSolder, F.Cu at (2.50, 23.5)
- added C201: 10uF, Capacitor_SMD:C_0402_1005Metric_Pad0.74x0.62mm_HandSolder, F.Cu at (120.7, 68.8)
- added C202: 0.1uF, Capacitor_SMD:C_0603_1608Metric_Pad1.08x0.95mm_HandSolder, F.Cu at (116.1, 87.8)
- added C203: 0.1uF, Capacitor_SMD:C_0603_1608Metric_Pad1.08x0.95mm_HandSolder, F.Cu at (21.5, 0.76)
- added C204: 0.1uF, Capacitor_SMD:C_0603_1608Metric_Pad1.08x0.95mm_HandSolder, F.Cu at (21.5, 3.27)
- added C205: 0.1uF, Capacitor_SMD:C_0603_1608Metric_Pad1.08x0.95mm_HandSolder, F.Cu at (21.5, 5.78)
- added C206: 0.1uF, Capacitor_SMD:C_0603_1608Metric_Pad1.08x0.95mm_HandSolder, F.Cu at (21.5, 8.29)
- added C207: 10nF, Capacitor_SMD:C_0402_1005Metric_Pad0.74x0.62mm_HandSolder, F.Cu at (120.7, 74.7)
- added C208: 10nF, Capacitor_SMD:C_0402_1005Metric_Pad0.74x0.62mm_HandSolder, F.Cu at (25.3, 3.44)
- added C209: 10uF, Capacitor_SMD:C_0402_1005Metric_Pad0.74x0.62mm_HandSolder, F.Cu at (25.3, 5.41)
- added C210: 1uF, Capacitor_SMD:C_0201_0603Metric_Pad0.64x0.40mm_HandSolder, F.Cu at (116.1, 84.3)
- added C211: 1uF, Capacitor_SMD:C_0201_0603Metric_Pad0.64x0.40mm_HandSolder, F.Cu at (25.1, 7.26)
- added C212: 0.1uF, Capacitor_SMD:C_0603_1608Metric_Pad1.08x0.95mm_HandSolder, F.Cu at (21.5, 10.8)
- added C213: 0.1uF, Capacitor_SMD:C_0603_1608Metric_Pad1.08x0.95mm_HandSolder, F.Cu at (21.5, 13.3)
- added C214: 10uF, Capacitor_SMD:C_0402_1005Metric_Pad0.74x0.62mm_HandSolder, F.Cu at (120.7, 76.7)
- added C8: 470nF, Capacitor_SMD:C_0201_0603Metric_Pad0.64x0.40mm_HandSolder, F.Cu at (13.7, 25.3)
- added C801: 100uF, Capacitor_SMD:C_0805_2012Metric_Pad1.18x1.45mm_HandSolder, F.Cu at (31.7, 70.4)
- added C802: 10uF, Capacitor_SMD:C_0402_1005Metric_Pad0.74x0.62mm_HandSolder, F.Cu at (39.8, 65.1)
- added C803: 0.1uF, Capacitor_SMD:C_0603_1608Metric_Pad1.08x0.95mm_HandSolder, F.Cu at (6.42, 0.76)
- added C804: 10uF, Capacitor_SMD:C_0402_1005Metric_Pad0.74x0.62mm_HandSolder, F.Cu at (5.86, 10.5)
- added C805: 0.1uF, Capacitor_SMD:C_0603_1608Metric_Pad1.08x0.95mm_HandSolder, F.Cu at (6.42, 3.27)
- added C806: 22uF, Capacitor_SMD:C_0603_1608Metric_Pad1.08x0.95mm_HandSolder, F.Cu at (6.42, 5.78)
- added C807: 22uF, Capacitor_SMD:C_0603_1608Metric_Pad1.08x0.95mm_HandSolder, F.Cu at (6.42, 8.29)
- added C808: 22uF, Capacitor_SMD:C_0603_1608Metric_Pad1.08x0.95mm_HandSolder, F.Cu at (10.8, 0.76)
- added C809: 22uF, Capacitor_SMD:C_0603_1608Metric_Pad1.08x0.95mm_HandSolder, F.Cu at (10.8, 3.27)
- added C810: 10uF, Capacitor_SMD:C_0402_1005Metric_Pad0.74x0.62mm_HandSolder, F.Cu at (5.86, 12.5)
- added C811: 0.1uF, Capacitor_SMD:C_0603_1608Metric_Pad1.08x0.95mm_HandSolder, F.Cu at (10.8, 5.78)
- added C812: 0.1uF, Capacitor_SMD:C_0603_1608Metric_Pad1.08x0.95mm_HandSolder, F.Cu at (10.8, 8.29)
- added C813: 1uF, Capacitor_SMD:C_0402_1005Metric_Pad0.74x0.62mm_HandSolder, F.Cu at (5.86, 14.5)
- added C814: 1uF, Capacitor_SMD:C_0402_1005Metric_Pad0.74x0.62mm_HandSolder, F.Cu at (5.86, 16.4)
- added C815: 0.1uF, Capacitor_SMD:C_0603_1608Metric_Pad1.08x0.95mm_HandSolder, F.Cu at (15.1, 0.76)
- added C816: 10uF, Capacitor_SMD:C_0402_1005Metric_Pad0.74x0.62mm_HandSolder, F.Cu at (5.86, 18.4)
- added C817: 0.1uF, Capacitor_SMD:C_0603_1608Metric_Pad1.08x0.95mm_HandSolder, F.Cu at (15.1, 3.27)
- added C818: 22uF, Capacitor_SMD:C_0603_1608Metric_Pad1.08x0.95mm_HandSolder, F.Cu at (15.1, 5.78)
- added C819: 22uF, Capacitor_SMD:C_0603_1608Metric_Pad1.08x0.95mm_HandSolder, F.Cu at (15.1, 8.29)
- added IC701: IP4220CZ6, Package_SO:SC-74-6_1.5x2.9mm_P0.95mm, F.Cu at (117.7, 105.5)
- added J10: EFM32_PinHeader_PortE, Connector_PinHeader_1.00mm:PinHeader_2x06_P1.00mm_Vertical, F.Cu at (109.8, 70.2)
- added J11: EFM32_PinHeader_PortE, Connector_PinHeader_1.00mm:PinHeader_2x06_P1.00mm_Vertical, F.Cu at (66.0, 73.3)
- added J12: EFM32_PinHeader_PortE, Connector_PinHeader_1.00mm:PinHeader_2x06_P1.00mm_Vertical, F.Cu at (103.4, 59.2)
- added J13: EFM32_PinHeader_PortE, Connector_PinHeader_1.00mm:PinHeader_2x06_P1.00mm_Vertical, F.Cu at (116.3, 59.2)
- added J14: Conn_02x10_Counter_Clockwise, Connector_PinHeader_1.00mm:PinHeader_2x10_P1.00mm_Vertical, F.Cu at (181.8, 86.6)
- added J201: Conn_ARM_JTAG_SWD_20, Connector_PinHeader_1.00mm:PinHeader_2x10_P1.00mm_Vertical, F.Cu at (116.4, 69.4)
- added J701: USB3_B_Micro, Connector_USB:USB_Micro-B_Wuerth_629105150521_CircularHoles, F.Cu at (108.1, 120.0)
- added J801: Conn_02x05_Odd_Even, Connector_PinHeader_2.00mm:PinHeader_2x05_P2.00mm_Vertical, F.Cu at (46.6, 66.1)
- added J802: Jack-DC, Connector_BarrelJack:BarrelJack_CUI_PJ-063AH_Horizontal_CircularHoles, F.Cu at (24.0, 82.5)
- added J803: USB_B_Micro, Connector_USB:USB_Micro-B_Wuerth_629105150521_CircularHoles, F.Cu at (16.0, 51.1)
- added L801: 1.5uH, Inductor_SMD:L_0805_2012Metric_Pad1.15x1.40mm_HandSolder, F.Cu at (31.0, 52.0)
- added L802: 1.5uH, Inductor_SMD:L_0805_2012Metric_Pad1.15x1.40mm_HandSolder, F.Cu at (31.0, 55.0)
- added R19: 100R, Resistor_SMD:R_0201_0603Metric_Pad0.64x0.40mm_HandSolder, F.Cu at (239.0, 104.2)
- added R19: 100k, Resistor_SMD:R_0805_2012Metric_Pad1.20x1.40mm_HandSolder, F.Cu at (83.0, 99.0)
- added R201: 100K, Resistor_SMD:R_0805_2012Metric_Pad1.20x1.40mm_HandSolder, F.Cu at (26.0, 0.97)
- added R801: 30.1K, Resistor_SMD:R_0805_2012Metric_Pad1.20x1.40mm_HandSolder, F.Cu at (1.88, 0.97)
- added R802: 22.1K, Resistor_SMD:R_0805_2012Metric_Pad1.20x1.40mm_HandSolder, F.Cu at (1.88, 3.92)
- added R803: 22.1K, Resistor_SMD:R_0805_2012Metric_Pad1.20x1.40mm_HandSolder, F.Cu at (1.88, 6.88)
- added R804: 100K, Resistor_SMD:R_0805_2012Metric_Pad1.20x1.40mm_HandSolder, F.Cu at (1.88, 9.82)
- added R805: 22.1K, Resistor_SMD:R_0805_2012Metric_Pad1.20x1.40mm_HandSolder, F.Cu at (1.88, 12.8)
- added R806: 73.2K, Resistor_SMD:R_0805_2012Metric_Pad1.20x1.40mm_HandSolder, F.Cu at (1.88, 15.7)
- added R807: 100k, Resistor_SMD:R_0805_2012Metric_Pad1.20x1.40mm_HandSolder, F.Cu at (35.8, 52.0)
- added SW801: SW_DPDT_x2, Button_Switch_THT:SW_E-Switch_EG2219_DPDT_Angled, F.Cu at (16.5, 63.0)
- added U201: EFM32GG11B420F2048GQ100, Package_QFP:TQFP-100_14x14mm_P0.5mm, F.Cu at (80.5, 77.0)
- added U202: IS62WVS2568FBLL-20NLI, Package_SO:SOIC-8_3.9x4.9mm_P1.27mm, F.Cu at (93.9, 84.6)
- added Y201: 48MHz, Crystal:Crystal_SMD_2016-4Pin_2.0x1.6mm, F.Cu at (100.0, 86.2)
- C29: value 0.1uF -> 100uF; footprint Capacitor_SMD:C_0201_0603Metric_Pad0.64x0.40mm_HandSolder -> Capacitor_SMD:C_1210_3225Metric_Pad1.33x2.70mm_HandSolder
- C60, C62: footprint Capacitor_SMD:C_0402_1005Metric_Pad0.74x0.62mm_HandSolder -> Capacitor_SMD:C_0805_2012Metric_Pad1.18x1.45mm_HandSolder
- C64, C76: footprint Capacitor_SMD:C_0201_0603Metric_Pad0.64x0.40mm_HandSolder -> Capacitor_SMD:C_0402_1005Metric_Pad0.74x0.62mm_HandSolder
- C68: value 100n -> 100nF
- C69: footprint Capacitor_SMD:C_0402_1005Metric_Pad0.74x0.62mm_HandSolder -> Capacitor_SMD:C_0201_0603Metric_Pad0.64x0.40mm_HandSolder
- IC2: moved to F.Cu
- J6: footprint Connector_PinHeader_2.54mm:PinHeader_2x06_P2.54mm_Vertical_SMD -> Connector_PinHeader_1.00mm:PinHeader_2x06_P1.00mm_Vertical
- R21: footprint Resistor_SMD:R_0805_2012Metric_Pad1.20x1.40mm_HandSolder -> Resistor_SMD:R_1206_3216Metric_Pad1.30x1.75mm_HandSolder
- SW1: footprint Button_Switch_SMD:SW_DIP_SPSTx01_Slide_6.7x4.1mm_W8.61mm_P2.54mm_LowProfile -> Button_Switch_SMD:SW_Push_1P1T_NO_CK_PTS125Sx43PSMTR
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Connections:
- net /MCU EFM32GG11B420/USB3_micro_ab/VBUS renamed VBUS
- net HDMI_TX1N renamed HDMI_TX1_N
- net HDMI_TX1P renamed HDMI_TX1_P
- net HDMI_TX2N renamed HDMI_TX2_N
- net HDMI_TX2P renamed HDMI_TX2_P
- C103 pad 2: +3V3 -> +3.3V
- C28 pad 1: +3V3 -> +3.3V
- C30 pad 1: +3V3 -> +3.3V
- C31 pad 1: +3V3 -> +3.3V
- C32 pad 1: +3V3 -> +3.3V
- C33 pad 1: +3V3 -> +3.3V
- C34 pad 1: +3V3 -> +3.3V
- C35 pad 1: +3V3 -> +3.3V
- C36 pad 1: +3V3 -> +3.3V
- C37 pad 1: +3V3 -> +3.3V
- C38 pad 1: +3V3 -> +3.3V
- C39 pad 1: +3V3 -> +3.3V
- C40 pad 1: +3V3 -> +3.3V
- C41 pad 1: +3V3 -> +3.3V
- C42 pad 1: +3V3 -> +3.3V
- C43 pad 1: +3V3 -> +3.3V
- C44 pad 1: +3V3 -> +3.3V
- C45 pad 1: +3V3 -> +3.3V
- C80 pad 1: +3V3 -> +3.3V
- C81 pad 1: +3V3 -> +3.3V
- C82 pad 1: +3V3 -> +3.3V
- C83 pad 1: +3V3 -> +3.3V
- C87 pad 1: +3V3 -> +3.3V
- C88 pad 1: +3V3 -> +3.3V
- C89 pad 1: +3V3 -> +3.3V
- C90 pad 1: +3V3 -> +3.3V
- C91 pad 1: +3V3 -> +3.3V
- C92 pad 1: +3V3 -> +3.3V
- C93 pad 1: +3V3 -> +3.3V
- J1 pad 2: +3V3 -> +3.3V
- J7 pad 10: HDMI_CLKP -> HDMI_CLK_P
- J7 pad 12: HDMI_CLKN -> HDMI_CLK_N
- J7 pad 7: HDMI_TX0P -> HDMI_TX0_P
- J7 pad 9: HDMI_TX0N -> HDMI_TX0_N
- R29 pad 1: +3V3 -> +3.3V
- R30 pad 1: +3V3 -> +3.3V
- R34 pad 2: +3V3 -> +3.3V
- R35 pad 2: +3V3 -> +3.3V
- R36 pad 2: +3V3 -> +3.3V
- R37 pad 2: +3V3 -> +3.3V
- R38 pad 1: +3V3 -> +3.3V
- U1 pad A17: +3V3 -> +3.3V
- U1 pad AA10: unconnected-(U1A-IO_L9P_T1_DQS_13-PadAA10) -> Net-(J14-Pin_7)
- U1 pad AA11: unconnected-(U1A-IO_L9N_T1_DQS_13-PadAA11) -> Net-(J14-Pin_8)
- U1 pad AA13: /MCU EFM32GG11B420/EBI_REn -> /MCU EFM32GG11B420/QSPI0_DQS
- U1 pad AA14: /FPGA Artix-7 100T 1FGG484C/EBI_A22 -> /FPGA Artix-7 100T 1FGG484C/QSPI0_DQ7
- U1 pad AA15: /FPGA Artix-7 100T 1FGG484C/EBI_A19 -> /FPGA Artix-7 100T 1FGG484C/QSPI0_DQ4
- U1 pad AA17: +3V3 -> +3.3V
- U1 pad AA9: unconnected-(U1A-IO_L8P_T1_13-PadAA9) -> Net-(J14-Pin_5)
- U1 pad AB10: unconnected-(U1A-IO_L8N_T1_13-PadAB10) -> Net-(J14-Pin_6)
- U1 pad AB11: unconnected-(U1A-IO_L7P_T1_13-PadAB11) -> Net-(J14-Pin_3)
- U1 pad AB12: unconnected-(U1A-IO_L7N_T1_13-PadAB12) -> Net-(J14-Pin_4)
- U1 pad AB13: /MCU EFM32GG11B420/EBI_BL0 -> /MCU EFM32GG11B420/QSPI0_SCLK
- U1 pad AB14: +3V3 -> +3.3V
- U1 pad AB15: /FPGA Artix-7 100T 1FGG484C/EBI_A20 -> /FPGA Artix-7 100T 1FGG484C/QSPI0_DQ5
- U1 pad B14: +3V3 -> +3.3V
- U1 pad C14: HDMI_CLKP -> HDMI_TX0_P
- U1 pad C15: HDMI_CLKN -> HDMI_TX0_N
- U1 pad C21: +3V3 -> +3.3V
- U1 pad D18: +3V3 -> +3.3V
- U1 pad E13: HDMI_TX0P -> HDMI_CLK_P
- U1 pad E14: HDMI_TX0N -> HDMI_CLK_N
- U1 pad E15: +3V3 -> +3.3V
- U1 pad F21: /MCU EFM32GG11B420/EBI_ARDY -> unconnected-(U1B-IO_25_16-PadF21)
- U1 pad F22: +3V3 -> +3.3V
- U1 pad G13: /FPGA Artix-7 100T 1FGG484C/EBI_A2 -> unconnected-(U1B-IO_L1N_T0_AD0N_15-PadG13)
- U1 pad G15: /FPGA Artix-7 100T 1FGG484C/EBI_A3 -> unconnected-(U1B-IO_L2P_T0_AD8P_15-PadG15)
- U1 pad G16: /FPGA Artix-7 100T 1FGG484C/EBI_A4 -> unconnected-(U1B-IO_L2N_T0_AD8N_15-PadG16)
- U1 pad G17: /FPGA Artix-7 100T 1FGG484C/EBI_A7 -> unconnected-(U1B-IO_L4P_T0_15-PadG17)
- U1 pad G18: /FPGA Artix-7 100T 1FGG484C/EBI_A8 -> unconnected-(U1B-IO_L4N_T0_15-PadG18)
- U1 pad G19: +3V3 -> +3.3V
- U1 pad G20: /FPGA Artix-7 100T 1FGG484C/EBI_A16 -> unconnected-(U1B-IO_L8N_T1_AD10N_15-PadG20)
- U1 pad H13: /FPGA Artix-7 100T 1FGG484C/EBI_A1 -> unconnected-(U1B-IO_L1P_T0_AD0P_15-PadH13)
- U1 pad H14: /FPGA Artix-7 100T 1FGG484C/EBI_A6 -> unconnected-(U1B-IO_L3N_T0_DQS_AD1N_15-PadH14)
- U1 pad H15: /FPGA Artix-7 100T 1FGG484C/EBI_A10 -> unconnected-(U1B-IO_L5N_T0_AD9N_15-PadH15)
- U1 pad H16: +3V3 -> +3.3V
- U1 pad H17: /FPGA Artix-7 100T 1FGG484C/EBI_A11 -> unconnected-(U1B-IO_L6P_T0_15-PadH17)
- U1 pad H18: /FPGA Artix-7 100T 1FGG484C/EBI_A12 -> unconnected-(U1B-IO_L6N_T0_VREF_15-PadH18)
- U1 pad H19: /FPGA Artix-7 100T 1FGG484C/EBI_A24 -> unconnected-(U1B-IO_L12N_T1_MRCC_15-PadH19)
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Routing:
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- added copper zone on In2.Cu, net +3.3V
- added copper zone on In1.Cu, net GND
Other:
- board outline added: 270 x 130 mm

Commit message: more pcb routing
Parts:
- removed C54: 10uF, Capacitor_SMD:C_0402_1005Metric_Pad0.74x0.62mm_HandSolder
- removed C55: 10nF, Capacitor_SMD:C_0402_1005Metric_Pad0.74x0.62mm_HandSolder
- removed C90, C91, C92, C93: 470nF, Capacitor_SMD:C_0201_0603Metric_Pad0.64x0.40mm_HandSolder
- removed J701: USB3_B_Micro, Connector_USB:USB_Micro-B_Wuerth_629105150521_CircularHoles
- removed the R19 at (83.0, 99.0)
- added C25: 47uF, Capacitor_SMD:C_1210_3225Metric_Pad1.33x2.70mm_HandSolder, F.Cu at (229.6, 125.9)
- added C46: 470nF, Capacitor_SMD:C_0201_0603Metric_Pad0.64x0.40mm_HandSolder, B.Cu at (204.4, 114.2)
- added C47: 470nF, Capacitor_SMD:C_0201_0603Metric_Pad0.64x0.40mm_HandSolder, B.Cu at (199.4, 111.9)
- added C48: 470nF, Capacitor_SMD:C_0201_0603Metric_Pad0.64x0.40mm_HandSolder, B.Cu at (199.7, 116.1)
- added C49: 470nF, Capacitor_SMD:C_0201_0603Metric_Pad0.64x0.40mm_HandSolder, B.Cu at (209.4, 113.5)
- added C60: 22uF, Capacitor_SMD:C_0402_1005Metric_Pad0.74x0.62mm_HandSolder, F.Cu at (39.8, 124.7)
- added C61: 100uF, Capacitor_SMD:C_1210_3225Metric_Pad1.33x2.70mm_HandSolder, F.Cu at (51.2, 110.5)
- added C62: 22uF, Capacitor_SMD:C_0402_1005Metric_Pad0.74x0.62mm_HandSolder, F.Cu at (38.0, 124.7)
- added C63: 10uF, Capacitor_SMD:C_0402_1005Metric_Pad0.74x0.62mm_HandSolder, F.Cu at (53.8, 110.4)
- added C64: 0.1uF, Capacitor_SMD:C_0201_0603Metric_Pad0.64x0.40mm_HandSolder, F.Cu at (55.4, 110.3)
- added C65: 10uF, Capacitor_SMD:C_0402_1005Metric_Pad0.74x0.62mm_HandSolder, F.Cu at (44.0, 118.7)
- added C66: 100nF, Capacitor_SMD:C_0201_0603Metric_Pad0.64x0.40mm_HandSolder, F.Cu at (48.0, 118.5)
- added C67: 10uF, Capacitor_SMD:C_0402_1005Metric_Pad0.74x0.62mm_HandSolder, F.Cu at (67.0, 105.3)
- added C68: 100n, Capacitor_SMD:C_0201_0603Metric_Pad0.64x0.40mm_HandSolder, F.Cu at (56.4, 119.1)
- added C69: 3.3nF, Capacitor_SMD:C_0402_1005Metric_Pad0.74x0.62mm_HandSolder, F.Cu at (67.6, 102.1)
- added C70: 1uF, Capacitor_SMD:C_0201_0603Metric_Pad0.64x0.40mm_HandSolder, F.Cu at (73.6, 102.1)
- added C71: 1uF, Capacitor_SMD:C_0201_0603Metric_Pad0.64x0.40mm_HandSolder, F.Cu at (68.6, 123.3)
- added C72: 100nF, Capacitor_SMD:C_0201_0603Metric_Pad0.64x0.40mm_HandSolder, F.Cu at (55.8, 102.3)
- added C73: 100nF, Capacitor_SMD:C_0201_0603Metric_Pad0.64x0.40mm_HandSolder, F.Cu at (68.4, 118.7)
- added C74: 10uF, Capacitor_SMD:C_0402_1005Metric_Pad0.74x0.62mm_HandSolder, F.Cu at (67.8, 115.3)
- added C75: 22uF, Capacitor_SMD:C_0402_1005Metric_Pad0.74x0.62mm_HandSolder, F.Cu at (49.8, 102.3)
- added C76: 100nF, Capacitor_SMD:C_0201_0603Metric_Pad0.64x0.40mm_HandSolder, F.Cu at (69.0, 115.1)
- added C77: 22uF, Capacitor_SMD:C_0402_1005Metric_Pad0.74x0.62mm_HandSolder, F.Cu at (48.2, 102.3)
- added C78: 22u, Capacitor_SMD:C_0402_1005Metric_Pad0.74x0.62mm_HandSolder, F.Cu at (76.5, 119.9)
- added C79: 22u, Capacitor_SMD:C_0402_1005Metric_Pad0.74x0.62mm_HandSolder, F.Cu at (75.1, 119.9)
- added J3: USB_B_Micro, Connector_USB:USB_Micro-B_GCT_USB3076-30-A, F.Cu at (147.0, 137.9)
- added J4: USB_B_Micro, Connector_USB:USB_Micro-B_Wuerth_629105150521_CircularHoles, F.Cu at (32.8, 119.5)
- added J5: Jack-DC, Connector_BarrelJack:BarrelJack_CUI_PJ-063AH_Horizontal_CircularHoles, F.Cu at (37.2, 102.4)
- added L1: 1.5uH, Inductor_SMD:L_0805_2012Metric_Pad1.15x1.40mm_HandSolder, F.Cu at (40.4, 120.1)
- added L2: 1.5uH, Inductor_SMD:L_0805_2012Metric_Pad1.15x1.40mm_HandSolder, F.Cu at (53.0, 101.9)
- added L3: 2.2uH, Inductor_SMD:L_0805_2012Metric_Pad1.15x1.40mm_HandSolder, F.Cu at (71.0, 119.1)
- added R20: 30.1k, Resistor_SMD:R_0805_2012Metric_Pad1.20x1.40mm_HandSolder, F.Cu at (42.6, 125.1)
- added R20: 10k, Resistor_SMD:R_0805_2012Metric_Pad1.20x1.40mm_HandSolder, B.Cu at (190.3, 123.7)
- added R21: 10k, Resistor_SMD:R_0805_2012Metric_Pad1.20x1.40mm_HandSolder, F.Cu at (191.5, 126.1)
- added R21: 22.1k, Resistor_SMD:R_0805_2012Metric_Pad1.20x1.40mm_HandSolder, F.Cu at (45.2, 127.3)
- added R22: 21.3k, Resistor_SMD:R_0805_2012Metric_Pad1.20x1.40mm_HandSolder, F.Cu at (68.8, 105.3)
- added R23: 22.1k, Resistor_SMD:R_0805_2012Metric_Pad1.20x1.40mm_HandSolder, F.Cu at (71.8, 105.3)
- added R23: 4.7k, Resistor_SMD:R_0603_1608Metric_Pad0.98x0.95mm_HandSolder, B.Cu at (215.8, 100.9)
- added R24: 4.7k, Resistor_SMD:R_0603_1608Metric_Pad0.98x0.95mm_HandSolder, F.Cu at (154.0, 100.4)
- added R24: 100k, Resistor_SMD:R_0805_2012Metric_Pad1.20x1.40mm_HandSolder, F.Cu at (71.8, 100.7)
- added R25: 100k, Resistor_SMD:R_0805_2012Metric_Pad1.20x1.40mm_HandSolder, F.Cu at (71.0, 124.1)
- added R26: 73.2k, Resistor_SMD:R_0805_2012Metric_Pad1.20x1.40mm_HandSolder, F.Cu at (79.8, 120.5)
- added R27: 22.1k, Resistor_SMD:R_0805_2012Metric_Pad1.20x1.40mm_HandSolder, F.Cu at (79.8, 124.9)
- added SW2: SW_DPDT_x2, Button_Switch_SMD:SW_DPDT_CK_JS202011JCQN, F.Cu at (44.4, 110.3)
- added SW3: SW_DIP_x05, Connector_PinHeader_1.27mm:PinHeader_2x05_P1.27mm_Vertical, F.Cu at (81.1, 107.9)
- added U2: TPS54325_PWP_14, Footprints:PWP14_2P31X2P46, F.Cu at (60.9, 102.3)
- added U5: TPS54294PWP, Footprints:PWP16_2P31X2P46, F.Cu at (63.0, 119.9)
- C1, C100, C104, C105, C11, C112, C113, C17, C18, C2, C22, C23, C24, C25, C28, C3, C30, C31, C32, C33, C39, C4, C40, C41, C42, C43, C44, C45, C5, C6, C7, C8, C80, C81, C82, C83, R19, TP4, U202: moved to B.Cu
- C10, C19, C9: footprint Capacitor_SMD:C_1210_3225Metric_Pad1.33x2.70mm_HandSolder -> Capacitor_SMD:C_0603_1608Metric_Pad1.08x0.95mm_HandSolder; moved to B.Cu
- C106, C107, C108, C109, C110, C111: footprint Capacitor_SMD:C_01005_0402Metric_Pad0.57x0.30mm_HandSolder -> Capacitor_SMD:C_0201_0603Metric_Pad0.64x0.40mm_HandSolder; moved to B.Cu
- C12, C20, C21: footprint Capacitor_SMD:C_0805_2012Metric_Pad1.18x1.45mm_HandSolder -> Capacitor_SMD:C_0201_0603Metric_Pad0.64x0.40mm_HandSolder; moved to B.Cu
- C16: footprint Capacitor_SMD:C_1210_3225Metric_Pad1.33x2.70mm_HandSolder -> Capacitor_SMD:C_0805_2012Metric_Pad1.18x1.45mm_HandSolder; moved to B.Cu
- C26: value 0.1uF -> 4.7uF; footprint Capacitor_SMD:C_0201_0603Metric_Pad0.64x0.40mm_HandSolder -> Capacitor_SMD:C_0805_2012Metric_Pad1.18x1.45mm_HandSolder
- C27: value 100uF -> 4.7uF
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Connections:
- J6 pad 1: /MCU EFM32GG11B420/PE0_UART0_TX -> /MCU EFM32GG11B420/MCU_EXTIO_PC6
- J6 pad 10: /MCU EFM32GG11B420/PE_6 -> /MCU EFM32GG11B420/PE2_UART0_CTS
- J6 pad 12: /MCU EFM32GG11B420/PE_7 -> /MCU EFM32GG11B420/PE3_UART0_RTS
- J6 pad 3: /MCU EFM32GG11B420/PE1_UART0_RX -> /MCU EFM32GG11B420/MCU_EXTIO_PC7
- J6 pad 5: /MCU EFM32GG11B420/PE2_UART0_CTS -> /MCU EFM32GG11B420/PE_6
- J6 pad 6: /MCU EFM32GG11B420/MCU_EXTIO_PC6 -> /MCU EFM32GG11B420/PE0_UART0_TX
- J6 pad 7: /MCU EFM32GG11B420/PE3_UART0_RTS -> /MCU EFM32GG11B420/PE_7
- J6 pad 8: /MCU EFM32GG11B420/MCU_EXTIO_PC7 -> /MCU EFM32GG11B420/PE1_UART0_RX
- R10 pad 1: /FPGA Artix-7 100T 1FGG484C/VGA connector/VGA_B1 -> /FPGA Artix-7 100T 1FGG484C/VGA_B1
- R11 pad 1: /FPGA Artix-7 100T 1FGG484C/VGA connector/VGA_B3 -> /FPGA Artix-7 100T 1FGG484C/VGA_B3
- R12 pad 1: /FPGA Artix-7 100T 1FGG484C/VGA connector/VGA_G1 -> /FPGA Artix-7 100T 1FGG484C/VGA_G1
- R13 pad 1: /FPGA Artix-7 100T 1FGG484C/VGA connector/VGA_G3 -> /FPGA Artix-7 100T 1FGG484C/VGA_G3
- R14 pad 1: /FPGA Artix-7 100T 1FGG484C/VGA connector/VGA_R1 -> /FPGA Artix-7 100T 1FGG484C/VGA_R1
- R15 pad 1: /FPGA Artix-7 100T 1FGG484C/VGA connector/VGA_R3 -> /FPGA Artix-7 100T 1FGG484C/VGA_R3
- R17 pad 2: /FPGA Artix-7 100T 1FGG484C/VGA connector/VGA_HSync -> /FPGA Artix-7 100T 1FGG484C/VGA_HSync
- R18 pad 2: /FPGA Artix-7 100T 1FGG484C/VGA connector/VGA_VSync -> /FPGA Artix-7 100T 1FGG484C/VGA_VSync
- R39 pad 2: /MCU EFM32GG11B420/PF10 -> /MCU EFM32GG11B420/USB_D-
- R4 pad 1: /FPGA Artix-7 100T 1FGG484C/VGA connector/VGA_B0 -> /FPGA Artix-7 100T 1FGG484C/VGA_B0
- R40 pad 1: /MCU EFM32GG11B420/PF11 -> /MCU EFM32GG11B420/USB_D+
- R5 pad 1: /FPGA Artix-7 100T 1FGG484C/VGA connector/VGA_B2 -> /FPGA Artix-7 100T 1FGG484C/VGA_B2
- R6 pad 1: /FPGA Artix-7 100T 1FGG484C/VGA connector/VGA_G0 -> /FPGA Artix-7 100T 1FGG484C/VGA_G0
- R7 pad 1: /FPGA Artix-7 100T 1FGG484C/VGA connector/VGA_G2 -> /FPGA Artix-7 100T 1FGG484C/VGA_G2
- R8 pad 1: /FPGA Artix-7 100T 1FGG484C/VGA connector/VGA_R0 -> /FPGA Artix-7 100T 1FGG484C/VGA_R0
- R9 pad 1: /FPGA Artix-7 100T 1FGG484C/VGA connector/VGA_R2 -> /FPGA Artix-7 100T 1FGG484C/VGA_R2
- U1 pad A15: unconnected-(U1B-IO_L9P_T1_DQS_16-PadA15) -> /FPGA Artix-7 100T 1FGG484C/QSPI0_DQ6
- U1 pad A16: unconnected-(U1B-IO_L9N_T1_DQS_16-PadA16) -> /FPGA Artix-7 100T 1FGG484C/QSPI0_DQ4
- U1 pad A18: unconnected-(U1B-IO_L17P_T2_16-PadA18) -> /FPGA Artix-7 100T 1FGG484C/QSPI0_DQ2
- U1 pad A19: unconnected-(U1B-IO_L17N_T2_16-PadA19) -> /FPGA Artix-7 100T 1FGG484C/QSPI0_DQ3
- U1 pad A20: unconnected-(U1B-IO_L16N_T2_16-PadA20) -> HDMI_TX2_P
- U1 pad A21: unconnected-(U1B-IO_L21N_T3_DQS_16-PadA21) -> HDMI_TX2_N
- U1 pad AA1: /FPGA Artix-7 100T 1FGG484C/DDR3/DDR3_nRESET -> /FPGA Artix-7 100T 1FGG484C/DDR3/DDR3_DQ0
- U1 pad AA13: /MCU EFM32GG11B420/QSPI0_DQS -> unconnected-(U1A-IO_L3P_T0_DQS_13-PadAA13)
- U1 pad AA14: /FPGA Artix-7 100T 1FGG484C/QSPI0_DQ7 -> unconnected-(U1A-IO_L5N_T0_13-PadAA14)
- U1 pad AA15: /FPGA Artix-7 100T 1FGG484C/QSPI0_DQ4 -> unconnected-(U1A-IO_L4P_T0_13-PadAA15)
- U1 pad AA16: /FPGA Artix-7 100T 1FGG484C/QSPI0_DQ1 -> unconnected-(U1A-IO_L1N_T0_13-PadAA16)
- U1 pad AA18: /FPGA Artix-7 100T 1FGG484C/VGA connector/VGA_R2 -> unconnected-(U1A-IO_L17P_T2_A14_D30_14-PadAA18)
- U1 pad AA20: /FPGA Artix-7 100T 1FGG484C/QSPI0_DQ1 -> /FPGA Artix-7 100T 1FGG484C/VGA_B2
- U1 pad AA21: /FPGA Artix-7 100T 1FGG484C/QSPI0_DQ2 -> /FPGA Artix-7 100T 1FGG484C/VGA_G0
- U1 pad AA3: /FPGA Artix-7 100T 1FGG484C/DDR3/DDR3_UDQS_P -> /FPGA Artix-7 100T 1FGG484C/DDR3/DDR3_A8
- U1 pad AA5: /FPGA Artix-7 100T 1FGG484C/DDR3/DDR3_DQ14 -> /FPGA Artix-7 100T 1FGG484C/DDR3/DDR3_DQ6
- U1 pad AA8: /FPGA Artix-7 100T 1FGG484C/DDR3/DDR3_A6 -> /FPGA Artix-7 100T 1FGG484C/DDR3/DDR3_UDQS_P
- U1 pad AB1: /FPGA Artix-7 100T 1FGG484C/DDR3/DDR3_A13 -> /FPGA Artix-7 100T 1FGG484C/DDR3/DDR3_LDQS_P
- U1 pad AB13: /MCU EFM32GG11B420/QSPI0_SCLK -> unconnected-(U1A-IO_L3N_T0_DQS_13-PadAB13)
- U1 pad AB15: /FPGA Artix-7 100T 1FGG484C/QSPI0_DQ5 -> unconnected-(U1A-IO_L4N_T0_13-PadAB15)
- U1 pad AB16: /FPGA Artix-7 100T 1FGG484C/QSPI0_DQ2 -> unconnected-(U1A-IO_L2P_T0_13-PadAB16)
- U1 pad AB17: /FPGA Artix-7 100T 1FGG484C/QSPI0_DQ3 -> unconnected-(U1A-IO_L2N_T0_13-PadAB17)
- U1 pad AB18: /FPGA Artix-7 100T 1FGG484C/VGA connector/VGA_R3 -> unconnected-(U1A-IO_L17N_T2_A13_D29_14-PadAB18)
- U1 pad AB2: /FPGA Artix-7 100T 1FGG484C/DDR3/DDR3_A9 -> /FPGA Artix-7 100T 1FGG484C/DDR3/DDR3_LDQS_N
- U1 pad AB20: unconnected-(U1A-IO_L15N_T2_DQS_DOUT_CSO_B_14-PadAB20) -> /FPGA Artix-7 100T 1FGG484C/VGA_B3
- U1 pad AB21: unconnected-(U1A-IO_L10P_T1_D14_14-PadAB21) -> /FPGA Artix-7 100T 1FGG484C/VGA_B1
- U1 pad AB22: unconnected-(U1A-IO_L10N_T1_D15_14-PadAB22) -> /FPGA Artix-7 100T 1FGG484C/VGA_B0
- U1 pad AB3: /FPGA Artix-7 100T 1FGG484C/DDR3/DDR3_A2 -> /FPGA Artix-7 100T 1FGG484C/DDR3/DDR3_DQ4
- U1 pad AB5: /FPGA Artix-7 100T 1FGG484C/DDR3/DDR3_A0 -> /FPGA Artix-7 100T 1FGG484C/DDR3/DDR3_DQ1
- U1 pad AB6: /FPGA Artix-7 100T 1FGG484C/DDR3/DDR3_A10 -> /FPGA Artix-7 100T 1FGG484C/DDR3/DDR3_LDM
- U1 pad AB7: /FPGA Artix-7 100T 1FGG484C/DDR3/DDR3_A11 -> /FPGA Artix-7 100T 1FGG484C/DDR3/DDR3_DQ8
- U1 pad AB8: /FPGA Artix-7 100T 1FGG484C/DDR3/DDR3_A8 -> /FPGA Artix-7 100T 1FGG484C/DDR3/DDR3_DQ12
- U1 pad B15: unconnected-(U1B-IO_L7P_T1_16-PadB15) -> /MCU EFM32GG11B420/QSPI0_CS1
- U1 pad B17: unconnected-(U1B-IO_L11P_T1_SRCC_16-PadB17) -> /FPGA Artix-7 100T 1FGG484C/QSPI0_DQ0
- U1 pad B18: unconnected-(U1B-IO_L11N_T1_SRCC_16-PadB18) -> /FPGA Artix-7 100T 1FGG484C/QSPI0_DQ1
- U1 pad B21: unconnected-(U1B-IO_L21P_T3_DQS_16-PadB21) -> HDMI_CEC
- U1 pad B22: unconnected-(U1B-IO_L20N_T3_16-PadB22) -> HDMI_TX1_P
- U1 pad C14: HDMI_TX0_P -> unconnected-(U1B-IO_L3P_T0_DQS_16-PadC14)
- U1 pad C15: HDMI_TX0_N -> unconnected-(U1B-IO_L3N_T0_DQS_16-PadC15)
- U1 pad C17: unconnected-(U1B-IO_L12N_T1_MRCC_16-PadC17) -> /FPGA Artix-7 100T 1FGG484C/QSPI0_DQ5
- U1 pad C18: unconnected-(U1B-IO_L13P_T2_MRCC_16-PadC18) -> /FPGA Artix-7 100T 1FGG484C/QSPI0_DQ7
- U1 pad C22: unconnected-(U1B-IO_L20P_T3_16-PadC22) -> HDMI_TX1_N
- U1 pad D14: HDMI_CEC -> /MCU EFM32GG11B420/QSPI0_SCLK
- U1 pad D16: HDMI_SDA -> unconnected-(U1B-IO_L5N_T0_16-PadD16)
- U1 pad D17: unconnected-(U1B-IO_L12P_T1_MRCC_16-PadD17) -> /MCU EFM32GG11B420/QSPI0_DQS
- U1 pad D20: unconnected-(U1B-IO_L19P_T3_16-PadD20) -> HDMI_SCL
- U1 pad D22: unconnected-(U1B-IO_L22N_T3_16-PadD22) -> HDMI_TX0_P
- U1 pad E12: GND -> +1V0
- U1 pad E13: HDMI_CLK_P -> unconnected-(U1B-IO_L4P_T0_16-PadE13)
- U1 pad E14: HDMI_CLK_N -> unconnected-(U1B-IO_L4N_T0_16-PadE14)
- U1 pad E16: HDMI_SCL -> unconnected-(U1B-IO_L5P_T0_16-PadE16)
- U1 pad E17: HDMI_TX1_N -> unconnected-(U1B-IO_L2N_T0_16-PadE17)
- U1 pad E22: unconnected-(U1B-IO_L22P_T3_16-PadE22) -> HDMI_TX0_N
- U1 pad F13: HDMI_TX2_P -> unconnected-(U1B-IO_L1P_T0_16-PadF13)
- U1 pad F14: HDMI_TX2_N -> unconnected-(U1B-IO_L1N_T0_16-PadF14)
- U1 pad F15: HDMI_HPD -> unconnected-(U1B-IO_0_16-PadF15)
- U1 pad F16: HDMI_TX1_P -> unconnected-(U1B-IO_L2P_T0_16-PadF16)
- U1 pad F19: unconnected-(U1B-IO_L18P_T2_16-PadF19) -> HDMI_HPD
- U1 pad F20: unconnected-(U1B-IO_L18N_T2_16-PadF20) -> HDMI_SDA
- U1 pad G19: +3.3V -> unconnected-(U1B-VCCO_15-PadG19)
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Routing:
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- added copper zone on In4.Cu, net GND
- removed copper zone on In2.Cu, net +3.3V
Other:
- board size 270 x 130 mm -> 268.6 x 82.9 mm
